File: Ramyun/RamyunActionBoard.brd (EAGLE design)
At the start: 160 x 100 mm, 1 part

Commit message: update
Parts:
- added C1: (no value), GFE:C0603(1608)_HANDSOLDER
- added C2: 0.1uF, GFE:C0603(1608)_HANDSOLDER
- added D1, D2, D3, D4, D5, D6, D7, D8: (no value), GFE:DO-27
- added D9: MBR120, GFE:SOD-123
- added Q1: BC817-16LT1SMD, GFE:SOT23-BEC
- added R1, R2, R3, R4, R5, R6, R7, R8: 390, GFE:R0603(1608)_HANDSOLDER
- added R10, R11, R14, R15, R9: 4.7k, GFE:R0603(1608)_HANDSOLDER
- added R12, R13: 1k, GFE:R0603(1608)_HANDSOLDER
- added U1, U2, U3, U4, U5, U6, U7, U8: PVN012PBF, GFE:DIL06
- added U10, U9: MAX31856_ADAFRUIT, GFE:MAX31856_ADAFRUIT
- added U11: GPS_ADAFRUIT, GFE:GPS_ADAFRUIT
- added U12: BUZZER, GFE:PS1240
- moved MS1 14.9 mm to (11.4, -25.4), turned to 90 degrees
Connections:
- new net +3V3: MS1.2
- new net +5V: C2.1, D9.A, R12.2, U12.1
- new net BUZZER: R13.1
- new net GND_EXT1: D1.A, D2.A, D3.A, D4.A
- new net GND_EXT2: D5.A, D6.A, D7.A, D8.A
- new net N$1: R8.2, U8.1
- new net N$10: R2.1
- new net N$11: R3.1
- new net N$12: R4.1
- new net N$13: R5.1
- new net N$14: R6.1
- new net N$15: R7.1
- new net N$16: R8.1
- new net N$17: Q1.B, R13.2
- new net N$18: Q1.C, R12.1, U12.2
- new net N$19: MS1.15, R14.1
- new net N$2: R7.2, U7.1
- new net N$20: MS1.14, R15.1
- new net N$21: R14.2
- new net N$23: R15.2
- new net N$25: D1.C, U1.5
- new net N$26: D2.C, U2.5
- new net N$27: D3.C, U3.5
- new net N$28: D4.C, U4.5
- new net N$29: D5.C, U5.5
- new net N$3: R6.2, U6.1
- new net N$30: D6.C, U6.5
- new net N$31: D7.C, U7.5
- new net N$32: D8.C, U8.5
- new net N$4: R5.2, U5.1
- new net N$5: R4.2, U4.1
- new net N$6: R3.2, U3.1
- new net N$7: R2.2, U2.1
- new net N$8: R1.2, U1.1
- new net N$9: R1.1
- new net USB: D9.C, MS1.26
- new net V_EXT1: U1.4, U1.6, U2.4, U2.6, U3.4, U3.6, U4.4, U4.6
- new net V_EXT2: U5.4, U5.6, U6.4, U6.6, U7.4, U7.6, U8.4, U8.6
- net GND: now also C2.2, Q1.E, U1.2, U2.2, U3.2, U4.2, U5.2, U6.2, U7.2, U8.2
Other:
- board size 160 x 100 mm -> 133 x 133 mm

Commit message: update
Parts:
- removed C1: (no value), GFE:C0603(1608)_HANDSOLDER
- added JP1, JP2, JP3, JP4: JP2, GFE:JP2SMD0603
- added R16, R17, R18, R19: 4.7k, GFE:R0603(1608)_HANDSOLDER
Connections:
- removed net N$10: R2.1
- removed net N$11: R3.1
- removed net N$12: R4.1
- removed net N$13: R5.1
- removed net N$14: R6.1
- removed net N$15: R7.1
- removed net N$16: R8.1
- removed net N$21: R14.2
- removed net N$23: R15.2
- removed net N$9: R1.1
- new net 10: JP1.2, MS1.22
- new net 12: JP2.2, MS1.24
- new net GPS_PPS: JP3.1, R19.1
- new net GPS_RX: R14.2, U11.6
- new net GPS_TX: R15.2, U11.5
- new net HP_OUT: MS1.20
- new net MISO: R16.2, U10.5, U9.5
- new net MOSI: R17.2, U10.6, U9.6
- new net N$22: MS1.13, R16.1
- new net N$24: MS1.12, R17.1
- new net N$33: MS1.11, R18.1
- new net N$34: R19.2, U11.9
- new net OUT_A1: MS1.5, R8.1
- new net OUT_A2: MS1.6, R7.1
- new net OUT_A3: MS1.7, R6.1
- new net OUT_A4: MS1.8, R5.1
- new net OUT_B1: MS1.9, R4.1
- new net OUT_B2: MS1.10, R3.1
- new net OUT_B3: JP4.1, R2.1
- new net OUT_B4: MS1.19, R1.1
- new net SCK: R18.2, U10.4, U9.4
- new net SCL: JP4.2, MS1.18
- new net SCL_EXT: JP4.3
- new net SDA: JP3.2, MS1.17
- new net SDA_EXT: JP3.3
- new net SERVO_1: MS1.21
- new net SERVO_2: JP1.3
- new net SERVO_3: JP2.3
- new net TEMP1_CS: JP1.1, U9.7
- new net TEMP2_CS: JP2.1, U10.7
- net +3V3: now also U10.1, U11.8, U9.1
- net BUZZER: now also MS1.23
- net GND: now also U10.3, U11.7, U9.3

Commit message: update
Connections:
- new net N$10: R10.2
- new net N$11: R11.2
- new net N$9: R9.2
- net SERVO_1: now also R9.1
- net SERVO_2: now also R10.1
- net SERVO_3: now also R11.1
Changed lines of the file:
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@@
 <signal name="SERVO_2">
 <contactref element="JP1" pad="3"/>
+<contactref element="R10" pad="1"/>
+<wire x1="-253.77" y1="-429.26" x2="-215.78" y2="-278.13" width="0" layer="19" extent="1-1"/>
 </signal>
 <signal name="SERVO_3">
 <contactref element="JP2" pad="3"/>
+<contactref element="R11" pad="1"/>
+<wire x1="-253.77" y1="-433.07" x2="-215.78" y2="-284.48" width="0" layer="19" extent="1-1"/>
 </signal>
 <signal name="SDA">
@@
 <signal name="SERVO_1">
 <contactref element="MS1" pad="21"/>
+<contactref element="R9" pad="1"/>
+<wire x1="-10.16" y1="8.89" x2="-215.78" y2="-271.78" width="0" layer="19" extent="1-1"/>
+</signal>
+<signal name="N$9">
+<contactref element="R9" pad="2"/>
+</signal>
+<signal name="N$10">
+<contactref element="R10" pad="2"/>
+</signal>
+<signal name="N$11">
+<contactref element="R11" pad="2"/>
 </signal>
 </signals>

Commit message: outline
Other:
- board size 133 x 133 mm -> 135.2 x 135.2 mm
Changed lines of the file:
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@@
 <board>
 <plain>
-<wire x1="66.5" y1="0" x2="-66.5" y2="0" width="0" layer="20" curve="-180"/>
-<wire x1="-66.5" y1="0" x2="66.5" y2="0" width="0" layer="20" curve="-180"/>
+<wire x1="-21.28205" y1="-63.104040625" x2="-19.87408125" y2="-63.56151875" width="0.001" layer="20"/>
+<wire x1="-19.87408125" y1="-63.56151875" x2="-12.311190625" y2="-67.10206875" width="0.001" layer="20"/>
+<wire x1="-12.311190625" y1="-67.10206875" x2="-9.02705" y2="-67.62223125" width="0.001" layer="20"/>
+<wire x1="-9.02705" y1="-67.62223125" x2="-0.740209375" y2="-66.59201875" width="0.001" layer="20"/>
+<wire x1="-0.740209375" y1="-66.59201875" x2="0.740209375" y2="-66.59201875" width="0.001" layer="20"/>
+<wire x1="0.740209375" y1="-66.59201875" x2="9.02705" y2="-67.62223125" width="0.001" layer="20"/>
+<wire x1="9.02705" y1="-67.62223125" x2="12.311190625" y2="-67.10206875" width="0.001" layer="20"/>
+<wire x1="12.311190625" y1="-67.10206875" x2="19.87408125" y2="-63.56151875" width="0.001" layer="20"/>
+<wire x1="19.87408125" y1="-63.56151875" x2="21.28205" y2="-63.104040625" width="0.001" layer="20"/>
+<wire x1="21.28205" y1="-63.104040625" x2="29.48165" y2="-61.52305" width="0.001" layer="20"/>
+<wire x1="29.48165" y1="-61.52305" x2="32.444309375" y2="-60.0135" width="0.001" layer="20"/>
+<wire x1="32.444309375" y1="-60.0135" x2="38.542959375" y2="-54.309159375" width="0.001" layer="20"/>
+<wire x1="38.542959375" y1="-54.309159375" x2="39.74065" y2="-53.438990625" width="0.001" layer="20"/>
+<wire x1="39.74065" y1="-53.438990625" x2="47.050390625" y2="-49.40156875" width="0.001" layer="20"/>
+<wire x1="47.050390625" y1="-49.40156875" x2="49.40156875" y2="-47.050390625" width="0.001" layer="20"/>
+<wire x1="49.40156875" y1="-47.050390625" x2="53.438990625" y2="-39.74065" width="0.001" layer="20"/>
+<wire x1="53.438990625" y1="-39.74065" x2="54.309159375" y2="-38.542959375" width="0.001" layer="20"/>
+<wire x1="54.309159375" y1="-38.542959375" x2="60.0135" y2="-32.444309375" width="0.001" layer="20"/>
+<wire x1="60.0135" y1="-32.444309375" x2="61.52305" y2="-29.48165" width="0.001" layer="20"/>
+<wire x1="61.52305" y1="-29.48165" x2="63.104040625" y2="-21.28205" width="0.001" layer="20"/>
+<wire x1="63.104040625" y1="-21.28205" x2="63.56151875" y2="-19.87408125" width="0.001" layer="20"/>
+<wire x1="63.56151875" y1="-19.87408125" x2="67.10206875" y2="-12.311190625" width="0.001" layer="20"/>
+<wire x1="67.10206875" y1="-12.311190625" x2="67.62223125" y2="-9.02705" width="0.001" layer="20"/>
+<wire x1="67.62223125" y1="-9.02705" x2="66.59201875" y2="-0.740209375" width="0.001" layer="20"/>
+<wire x1="66.59201875" y1="-0.740209375" x2="66.59201875" y2="0.740209375" width="0.001" layer="20"/>
+<wire x1="66.59201875" y1="0.740209375" x2="67.62223125" y2="9.02705" width="0.001" layer="20"/>
+<wire x1="67.62223125" y1="9.02705" x2="67.10206875" y2="12.311190625" width="0.001" layer="20"/>
+<wire x1="67.10206875" y1="12.311190625" x2="63.56151875" y2="19.87408125" width="0.001" layer="20"/>
+<wire x1="63.56151875" y1="19.87408125" x2="63.104040625" y2="21.28205" width="0.001" layer="20"/>
+<wire x1="63.104040625" y1="21.28205" x2="61.52305" y2="29.48165" width="0.001" layer="20"/>
+<wire x1="61.52305" y1="29.48165" x2="60.0135" y2="32.444309375" width="0.001" layer="20"/>
+<wire x1="60.0135" y1="32.444309375" x2="54.309159375" y2="38.542959375" width="0.001" layer="20"/>
+<wire x1="54.309159375" y1="38.542959375" x2="53.438990625" y2="39.74065" width="0.001" layer="20"/>
+<wire x1="53.438990625" y1="39.74065" x2="49.40156875" y2="47.050390625" width="0.001" layer="20"/>
+<wire x1="49.40156875" y1="47.050390625" x2="47.050390625" y2="49.40156875" width="0.001" layer="20"/>
+<wire x1="47.050390625" y1="49.40156875" x2="39.74065" y2="53.438990625" width="0.001" layer="20"/>
+<wire x1="39.74065" y1="53.438990625" x2="38.542959375" y2="54.309159375" width="0.001" layer="20"/>
+<wire x1="38.542959375" y1="54.309159375" x2="32.444309375" y2="60.0135" width="0.001" layer="20"/>
+<wire x1="32.444309375" y1="60.0135" x2="29.48165" y2="61.52305" width="0.001" layer="20"/>
+<wire x1="29.48165" y1="61.52305" x2="21.28205" y2="63.104040625" width="0.001" layer="20"/>
+<wire x1="21.28205" y1="63.104040625" x2="19.87408125" y2="63.56151875" width="0.001" layer="20"/>
+<wire x1="19.87408125" y1="63.56151875" x2="12.311190625" y2="67.10206875" width="0.001" layer="20"/>
+<wire x1="12.311190625" y1="67.10206875" x2="9.02705" y2="67.62223125" width="0.001" layer="20"/>
+<wire x1="9.02705" y1="67.62223125" x2="0.740209375" y2="66.59201875" width="0.001" layer="20"/>
+<wire x1="0.740209375" y1="66.59201875" x2="-0.740209375" y2="66.59201875" width="0.001" layer="20"/>
+<wire x1="-0.740209375" y1="66.59201875" x2="-9.02705" y2="67.62223125" width="0.001" layer="20"/>
+<wire x1="-9.02705" y1="67.62223125" x2="-12.311190625" y2="67.10206875" width="0.001" layer="20"/>
+<wire x1="-12.311190625" y1="67.10206875" x2="-19.87408125" y2="63.56151875" width="0.001" layer="20"/>
+<wire x1="-19.87408125" y1="63.56151875" x2="-21.28205" y2="63.104040625" width="0.001" layer="20"/>
+<wire x1="-21.28205" y1="63.104040625" x2="-29.48165" y2="61.52305" width="0.001" layer="20"/>
+<wire x1="-29.48165" y1="61.52305" x2="-32.444309375" y2="60.0135" width="0.001" layer="20"/>
+<wire x1="-32.444309375" y1="60.0135" x2="-38.542959375" y2="54.309159375" width="0.001" layer="20"/>
+<wire x1="-38.542959375" y1="54.309159375" x2="-39.74065" y2="53.438990625" width="0.001" layer="20"/>
+<wire x1="-39.74065" y1="53.438990625" x2="-47.050390625" y2="49.40156875" width="0.001" layer="20"/>
+<wire x1="-47.050390625" y1="49.40156875" x2="-49.40156875" y2="47.050390625" width="0.001" layer="20"/>
+<wire x1="-49.40156875" y1="47.050390625" x2="-53.438990625" y2="39.74065" width="0.001" layer="20"/>
+<wire x1="-53.438990625" y1="39.74065" x2="-54.309159375" y2="38.542959375" width="0.001" layer="20"/>
+<wire x1="-54.309159375" y1="38.542959375" x2="-60.0135" y2="32.444309375" width="0.001" layer="20"/>
+<wire x1="-60.0135" y1="32.444309375" x2="-61.52305" y2="29.48165" width="0.001" layer="20"/>
+<wire x1="-61.52305" y1="29.48165" x2="-63.104040625" y2="21.28205" width="0.001" layer="20"/>
+<wire x1="-63.104040625" y1="21.28205" x2="-63.56151875" y2="19.87408125" width="0.001" layer="20"/>
+<wire x1="-63.56151875" y1="19.87408125" x2="-67.10206875" y2="12.311190625" width="0.001" layer="20"/>
+<wire x1="-67.10206875" y1="12.311190625" x2="-67.62223125" y2="9.02705" width="0.001" layer="20"/>
+<wire x1="-67.62223125" y1="9.02705" x2="-66.59201875" y2="0.740209375" width="0.001" layer="20"/>
+<wire x1="-66.59201875" y1="0.740209375" x2="-66.59201875" y2="-0.740209375" width="0.001" layer="20"/>
+<wire x1="-66.59201875" y1="-0.740209375" x2="-67.62223125" y2="-9.02705" width="0.001" layer="20"/>
+<wire x1="-67.62223125" y1="-9.02705" x2="-67.10206875" y2="-12.311190625" width="0.001" layer="20"/>
+<wire x1="-67.10206875" y1="-12.311190625" x2="-63.56151875" y2="-19.87408125" width="0.001" layer="20"/>
+<wire x1="-63.56151875" y1="-19.87408125" x2="-63.104040625" y2="-21.28205" width="0.001" layer="20"/>
+<wire x1="-63.104040625" y1="-21.28205" x2="-61.52305" y2="-29.48165" width="0.001" layer="20"/>
+<wire x1="-61.52305" y1="-29.48165" x2="-60.0135" y2="-32.444309375" width="0.001" layer="20"/>
+<wire x1="-60.0135" y1="-32.444309375" x2="-54.309159375" y2="-38.542959375" width="0.001" layer="20"/>
+<wire x1="-54.309159375" y1="-38.542959375" x2="-53.438990625" y2="-39.74065" width="0.001" layer="20"/>
+<wire x1="-53.438990625" y1="-39.74065" x2="-49.40156875" y2="-47.050390625" width="0.001" layer="20"/>
+<wire x1="-49.40156875" y1="-47.050390625" x2="-47.050390625" y2="-49.40156875" width="0.001" layer="20"/>
+<wire x1="-47.050390625" y1="-49.40156875" x2="-39.74065" y2="-53.438990625" width="0.001" layer="20"/>
+<wire x1="-39.74065" y1="-53.438990625" x2="-38.542959375" y2="-54.309159375" width="0.001" layer="20"/>
+<wire x1="-38.542959375" y1="-54.309159375" x2="-32.444309375" y2="-60.0135" width="0.001" layer="20"/>
+<wire x1="-32.444309375" y1="-60.0135" x2="-29.48165" y2="-61.52305" width="0.001" layer="20"/>
+<wire x1="-29.48165" y1="-61.52305" x2="-21.28205" y2="-63.104040625" width="0.001" layer="20"/>
 </plain>
 <attributes>

Commit message: update
Parts:
- added D10: MBR120, GFE:SOD-123
- added H1, H2, H3, H4: MOUNT-HOLE4.1, holes:4,1
- added Q2: NVF6P02, GFE:SOT223
- added S1: (no value), GFE:SKHLACA010
- added X1, X2, X3: 5267-03, GFE:5267-03
- added X10, X11, X12, X13, X14, X4, X5, X6, X7, X8, X9: 5267-02, GFE:5267-02
- moved U8 178.5 mm to (-47.0, 17.8), turned to 90 degrees
- moved U7 156.4 mm to (-47.0, 6.35), turned to 90 degrees
- moved U6 135.4 mm to (-47.0, -2.54), turned to 90 degrees
- moved U5 114.4 mm to (-47.0, -11.4), turned to 90 degrees
- moved U4 93.4 mm to (-47.0, -20.3), turned to 90 degrees
- moved U3 72.4 mm to (-47.0, -29.2), turned to 90 degrees
- moved U10 64.5 mm to (1.27, 24.1)
- moved U9 64.5 mm to (-25.4, 24.1)
- moved U11 63.5 mm to (0.00, -34.3), turned to 180 degrees
- moved U2 51.9 mm to (-47.0, -36.8), turned to 90 degrees
- moved U1 30.5 mm to (-47.0, -47.0), turned to 90 degrees
- moved MS1 27.9 mm to (0.00, 0.00), turned to 180 degrees
Connections:
- removed net USB: D9.C, MS1.26
- new net EXT_5V: Q2.2, Q2.4, X4.1
- new net LED1: MS1.25
- net +5V: now also Q2.3, X1.1, X2.1, X3.1; no longer D9.A
- net GND: now also Q2.1, X1.3, X2.3, X3.3, X4.2
- net GND_EXT1: now also X10.2, X5.2, X7.2, X8.2, X9.2
- net GND_EXT2: now also X11.2, X12.2, X13.2, X14.2, X6.2
- net N$10: now also X2.2
- net N$11: now also X3.2
- net N$25: now also X7.1
- net N$26: now also X8.1
- net N$27: now also X9.1
- net N$28: now also X10.1
- net N$29: now also X11.1
- net N$30: now also X12.1
- net N$31: now also X13.1
- net N$32: now also X14.1
- net N$9: now also X1.2
- net V_EXT1: now also X5.1
- net V_EXT2: now also X6.1

Commit message: layout almost done
Parts:
- removed D10: MBR120, GFE:SOD-123
- removed H3: MOUNT-HOLE4.1, holes:4,1
- removed S1: (no value), GFE:SKHLACA010
- added C1: (no value), adafruit:E3,5-8
- added JP5, JP6: M02PTH, berry:1X02
- added LOGO1: GRADEFREELOGO-20, GFE:GRADEFREELOGO-20
- added Q4: BC817-16LT1SMD, GFE:SOT23-BEC
- added R22, R23: 1k, GFE:R0603(1608)_HANDSOLDER
- added U13: NL17SZ17, GFE:SOT-553
- added X15: 5267-02, GFE:5267-02
- D1, D2, D3, D4, D5, D6, D7, D8: device GFE:DO-27 -> GFE:DO-27-VERTICAL
- R10, R11, R9: value 4.7k -> 390
- moved Q2 784.5 mm to (49.5, 17.8), turned to 180 degrees
- moved X14 756.4 mm to (-47.0, 39.4), turned to 90 degrees
- moved X13 729.9 mm to (-54.6, 29.2), turned to 90 degrees
- moved X12 704.4 mm to (-58.4, 19.1), turned to 90 degrees
- moved X11 679.3 mm to (-61.0, 8.89), turned to 90 degrees
- moved X6 655.5 mm to (-31.8, 50.8), turned to 90 degrees
- moved X10 647.6 mm to (-61.0, -8.89), turned to 90 degrees
- moved X4 634.4 mm to (58.4, 17.8), turned to 270 degrees
- moved X9 624.1 mm to (-58.4, -19.1), turned to 90 degrees
- moved X8 601.2 mm to (-54.6, -29.2), turned to 90 degrees
- moved X7 579.9 mm to (-47.0, -39.4), turned to 90 degrees
- moved X5 546.6 mm to (-31.8, -50.8), turned to 90 degrees
- moved X2 544.6 mm to (55.9, -25.4), turned to 270 degrees
- moved X3 543.9 mm to (47.0, -38.1), turned to 270 degrees
- moved X1 542.5 mm to (59.7, -12.7), turned to 270 degrees
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Connections:
- new net HP_SSR: U13.4, X15.1
- new net N$13: JP5.2, R23.2
- new net N$14: Q4.C, R23.1
- new net N$15: Q4.B, R22.2
- new net USB: D9.C, JP6.2, MS1.26
- net +5V: now also C1.+, D9.A, JP5.1, JP6.1, U13.5
- net GND: now also C1.-, Q4.E, U13.3, X15.2
- net HP_OUT: now also U13.2
- net LED1: now also R22.1
Other:
- board text added: "Project R"

Commit message: updated
Parts:
- removed JP6: M02PTH, berry:1X02
- added J1: (no value), SparkFun-Connectors:1X04
- added LED1: (no value), GFE:LED3MM
- added R20: 500, GFE:R0603(1608)_HANDSOLDER
- added X16: USB+SHIELD, GFE:USB-B-PTH
- moved D9 32.5 mm to (53.3, -7.62), turned to 0 degrees
- moved R16 11.7 mm to (-15.2, 15.2)
- moved R17 11.7 mm to (-12.7, 15.2)
- moved R18 11.7 mm to (-10.2, 15.2)
- moved MS1 3.81 mm to (-3.81, 0.00)
- moved R10 1.80 mm to (48.3, -26.7)
- moved X2 1.80 mm to (54.6, -26.7)
- moved R9 1.80 mm to (52.1, -14.0)
- moved R11 1.80 mm to (39.4, -39.4)
- moved X3 1.80 mm to (45.7, -39.4)
- moved X1 1.80 mm to (58.4, -14.0)
- moved C1 1.27 mm to (39.4, 17.8)
- turned D1 to 35 degrees
- turned D2 to 35 degrees
- turned D3 to 35 degrees
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Connections:
- removed net USB: D9.C, JP6.2, MS1.26
- new net D+: J1.3, X16.D+
- new net D-: J1.2, X16.D-
- new net N$12: D9.A, X16.VBUS
- new net N$16: LED1.A, R20.1
- new net STRUT_GND: X16.S1, X16.S2
- new net VBUS: D9.C, J1.1
- net +5V: now also MS1.26, R20.2; no longer D9.A, JP6.1
- net GND: now also J1.4, LED1.K, X16.GND
