File: Ramyun/RamyunActionBoard.brd (EAGLE design)
At the start: 135.2 x 135.2 mm, 77 parts, among them Q1 BC817-16LT1SMD, Q2 NVF6P02, Q4 BC817-16LT1SMD, U1 PVN012PBF, U10 MAX31856_ADAFRUIT, U11 GPS_ADAFRUIT, U12 BUZZER, U13 NL17SZ17, U2 PVN012PBF, U3 PVN012PBF, U4 PVN012PBF, U5 PVN012PBF, U6 PVN012PBF, U7 PVN012PBF, U8 PVN012PBF, U9 MAX31856_ADAFRUIT, X1 5267-03, X10 5267-02, X11 5267-02, X12 5267-02, X13 5267-02, X14 5267-02, X15 5267-02, X16 USB+SHIELD, X2 5267-03, X3 5267-03, X4 5267-02, X5 5267-02, X6 5267-02, X7 5267-02, X8 5267-02, X9 5267-02

Commit message: tired
Parts:
- removed Q4: BC817-16LT1SMD, GFE:SOT23-BEC
- removed R23: 1k, GFE:R0603(1608)_HANDSOLDER
- added H3: MOUNT-HOLE4.1, holes:4,1
- added Q3: NVF6P02, GFE:SOT223
- added R21: 390, GFE:R0603(1608)_HANDSOLDER
- C1: value (none) -> 0.1uF; device adafruit:E3,5-8 -> GFE:C0603(1608)_HANDSOLDER
- C2: value 0.1uF -> (none); device GFE:C0603(1608)_HANDSOLDER -> adafruit:E3,5-8
- D1: value (none) -> MBR120; device GFE:DO-27-VERTICAL -> GFE:SOD-123
- D9: value MBR120 -> (none); device GFE:SOD-123 -> GFE:DO-27-VERTICAL
- Q2: value NVF6P02 -> BC817-16LT1SMD; device GFE:SOT223 -> GFE:SOT23-BEC
- R10, R11, R4, R7, R8, R9: value 390 -> 4.7k
- R14: value 4.7k -> 500
- R15, R16, R17, R18, R19: value 4.7k -> 390
- R20: value 500 -> 390
- R22: value 1k -> 390
- R5, R6: value 390 -> 1k
- U1, U2: value PVN012PBF -> MAX31856_ADAFRUIT; device GFE:DIL06 -> GFE:MAX31856_ADAFRUIT
- U10, U9: value MAX31856_ADAFRUIT -> PVN012PBF; device GFE:MAX31856_ADAFRUIT -> GFE:DIL06
- U11: value GPS_ADAFRUIT -> PVN012PBF; device GFE:GPS_ADAFRUIT -> GFE:DIL06
- U12: value BUZZER -> PVN012PBF; device GFE:PS1240 -> GFE:DIL06
- U13: value NL17SZ17 -> PVN012PBF; device GFE:SOT-553 -> GFE:DIL06
- U3: value PVN012PBF -> NL17SZ17; device GFE:DIL06 -> GFE:SOT-553
- U4: value PVN012PBF -> GPS_ADAFRUIT; device GFE:DIL06 -> GFE:GPS_ADAFRUIT
- U5: value PVN012PBF -> BUZZER; device GFE:DIL06 -> GFE:PS1240
- X16: value USB+SHIELD -> 5267-02; device GFE:USB-B-PTH -> GFE:5267-02
- X4: value 5267-02 -> USB+SHIELD; device GFE:5267-02 -> GFE:USB-B-PTH
- moved X5 120.8 mm to (45.7, 41.9), turned to 270 degrees
- moved X16 105.7 mm to (-31.8, 50.8), turned to 90 degrees
- moved D9 101.7 mm to (-36.8, 39.4), turned to 35 degrees
- moved U3 98.6 mm to (40.6, 41.9), turned to 180 degrees
- moved X6 96.0 mm to (58.4, 17.8), turned to 270 degrees
- moved D1 95.6 mm to (53.3, -7.62), turned to 0 degrees
- moved X15 92.7 mm to (-47.0, 39.4), turned to 90 degrees
- moved U12 87.3 mm to (-33.0, 29.2), turned to 90 degrees
- moved R20 79.1 mm to (-30.5, 19.1), turned to 270 degrees
- moved U5 78.2 mm to (24.1, -36.8), turned to 180 degrees
- moved R1 75.5 mm to (52.1, -14.0), turned to 0 degrees
- moved R2 75.0 mm to (48.3, -26.7), turned to 0 degrees
- moved R3 72.7 mm to (39.4, -39.4), turned to 0 degrees
- moved R11 72.2 mm to (-6.35, 16.5), turned to 90 degrees
- moved R6 72.0 mm to (24.1, -27.9), turned to 0 degrees
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Connections:
- net +3V3: now also U1.1, U2.1, U4.8; no longer U10.1, U11.8, U9.1
- net +5V: now also C1.1, C2.+, Q3.3, R14.2, R6.2, U3.5, U5.1; no longer C1.+, C2.1, Q2.3, R12.2, R20.2, U12.1, U13.5
- net 10: now also JP3.2; no longer JP1.2
- net 12: now also JP4.2; no longer JP2.2
- net BUZZER: now also R5.1; no longer R13.1
- net D+: now also X4.D+; no longer X16.D+
- net D-: now also X4.D-; no longer X16.D-
- net EXT_5V: now also Q3.2, Q3.4, X6.1; no longer Q2.2, Q2.4, X4.1
- net GND: now also C1.2, C2.-, Q2.E, Q3.1, U1.3, U10.2, U11.2, U12.2, U13.2, U2.3, U3.3, U4.7, U9.2, X4.GND, X5.2, X6.2; no longer C1.-, C2.2, Q2.1, Q4.E, U1.2, U10.3, U11.7, U13.3, U2.2, U3.2, U4.2, U5.2, U9.3, X15.2, X16.GND, X4.2
- net GND_EXT1: now also D5.A, X11.2; no longer D1.A, X5.2
- net GND_EXT2: now also D9.A, X15.2, X16.2; no longer D5.A, X11.2, X6.2
- net GPS_PPS: now also JP1.1, R4.1; no longer JP3.1, R19.1
- net GPS_RX: now also R7.2, U4.6; no longer R14.2, U11.6
- net GPS_TX: now also R8.2, U4.5; no longer R15.2, U11.5
- net HP_OUT: now also U3.2; no longer U13.2
- net HP_SSR: now also U3.4, X5.1; no longer U13.4, X15.1
- net LED1: now also R12.1; no longer R22.1
- net MISO: now also R9.2, U1.5, U2.5; no longer R16.2, U10.5, U9.5
- net MOSI: now also R10.2, U1.6, U2.6; no longer R17.2, U10.6, U9.6
- net N$1: now also R22.2, U13.1; no longer R8.2, U8.1
- net N$10: now also R2.2; no longer R10.2
- net N$11: now also R3.2; no longer R11.2
- net N$12: now also D1.A, X4.VBUS; no longer D9.A, X16.VBUS
- net N$13: now also R13.2; no longer R23.2
- net N$14: now also Q2.C, R13.1; no longer Q4.C, R23.1
- net N$15: now also Q2.B, R12.2; no longer Q4.B, R22.2
- net N$16: now also R14.1; no longer R20.1
- net N$17: now also R5.2; no longer R13.2
- net N$18: now also R6.1, U5.2; no longer R12.1, U12.2
- net N$19: now also R7.1; no longer R14.1
- net N$2: now also R21.2, U12.1; no longer R7.2, U7.1
- net N$20: now also R8.1; no longer R15.1
- net N$22: now also R9.1; no longer R16.1
- net N$24: now also R10.1; no longer R17.1
- net N$25: now also D2.C, U6.5, X8.1; no longer D1.C, U1.5, X7.1
- net N$26: now also D3.C, U7.5, X9.1; no longer D2.C, U2.5, X8.1
- net N$27: now also D4.C, U8.5, X10.1; no longer D3.C, U3.5, X9.1
- net N$28: now also D5.C, U9.5, X11.1; no longer D4.C, U4.5, X10.1
- net N$29: now also D6.C, U10.5, X12.1; no longer D5.C, U5.5, X11.1
- net N$3: now also R20.2, U11.1; no longer R6.2, U6.1
- net N$30: now also D7.C, U11.5, X13.1; no longer D6.C, U6.5, X12.1
- net N$31: now also D8.C, U12.5, X14.1; no longer D7.C, U7.5, X13.1
- net N$32: now also D9.C, U13.5, X15.1; no longer D8.C, U8.5, X14.1
- net N$33: now also R11.1; no longer R18.1
- net N$34: now also R4.2, U4.9; no longer R19.2, U11.9
- net N$4: now also R19.2, U10.1; no longer R5.2, U5.1
- net N$5: now also R18.2, U9.1; no longer R4.2, U4.1
- net N$6: now also R17.2, U8.1; no longer R3.2, U3.1
- net N$7: now also R16.2, U7.1; no longer R2.2, U2.1
- net N$8: now also R15.2, U6.1; no longer R1.2, U1.1
- net N$9: now also R1.2; no longer R9.2
- net OUT_A1: now also R22.1; no longer R8.1
- net OUT_A2: now also R21.1; no longer R7.1
- net OUT_A3: now also R20.1; no longer R6.1
- net OUT_A4: now also R19.1; no longer R5.1
- net OUT_B1: now also R18.1; no longer R4.1
- net OUT_B2: now also R17.1; no longer R3.1
- net OUT_B3: now also JP2.1, R16.1; no longer JP4.1, R2.1
- net OUT_B4: now also R15.1; no longer R1.1
- net SCK: now also R11.2, U1.4, U2.4; no longer R18.2, U10.4, U9.4
- net SCL: now also JP2.2; no longer JP4.2
- net SCL_EXT: now also JP2.3; no longer JP4.3
- net SDA: now also JP1.2; no longer JP3.2
- net SDA_EXT: now also JP1.3; no longer JP3.3
- net SERVO_1: now also R1.1; no longer R9.1
- net SERVO_2: now also JP3.3, R2.1; no longer JP1.3, R10.1
- net SERVO_3: now also JP4.3, R3.1; no longer JP2.3, R11.1
- net STRUT_GND: now also X4.S1, X4.S2; no longer X16.S1, X16.S2
- net TEMP1_CS: now also JP3.1, U1.7; no longer JP1.1, U9.7
- net TEMP2_CS: now also JP4.1, U2.7; no longer JP2.1, U10.7
- net VBUS: now also D1.C; no longer D9.C
- net V_EXT1: now also U6.4, U6.6, U7.4, U7.6, U8.4, U8.6, U9.4, U9.6, X7.1; no longer U1.4, U1.6, U2.4, U2.6, U3.4, U3.6, U4.4, U4.6, X5.1
- net V_EXT2: now also U10.4, U10.6, U11.4, U11.6, U12.4, U12.6, U13.4, U13.6, X16.1; no longer U5.4, U5.6, U6.4, U6.6, U7.4, U7.6, U8.4, U8.6, X6.1
