File: Ramyun/RamyunActionBoard.sch (EAGLE design)
At the start: 1 part

Commit message: update
Parts:
- added C1: (no value), GFE:C0603(1608)_HAND
- added C2: 0.1uF, GFE:C0603(1608)_HAND
- added D1, D2, D3, D4, D5, D6, D7, D8: (no value), GFE:MBR5200VPTR-E1
- added D9: MBR120, GFE:MBR120
- added Q1: BC817-16LT1SMD, GFE:BC817-16LT1SMD
- added R1, R2, R3, R4, R5, R6, R7, R8: 390, GFE:R0603(1608)_HAND
- added R10, R11, R14, R15, R9: 4.7k, GFE:R0603(1608)_HAND
- added R12, R13: 1k, GFE:R0603(1608)_HAND
- added U1, U2, U3, U4, U5, U6, U7, U8: PVN012PBF, GFE:PVN012PBF
- added U10, U9: MAX31856_ADAFRUIT, GFE:MAX31856_ADAFRUIT
- added U11: GPS_ADAFRUIT, GFE:GPS_ADAFRUIT
- added U12: BUZZER, GFE:BUZZER
Connections:
- new net +3V3: MS1.3V
- new net +5V: C2.1, D9.A, R12.2, U12.P$1
- new net BUZZER: R13.1
- new net GND: C2.2, MS1.GND, Q1.E, U1.2, U2.2, U3.2, U4.2, U5.2, U6.2, U7.2, U8.2
- new net GND_EXT1: D1.A, D2.A, D3.A, D4.A
- new net GND_EXT2: D5.A, D6.A, D7.A, D8.A
- new net N$1: R8.2, U8.1
- new net N$10: R2.1
- new net N$11: R3.1
- new net N$12: R4.1
- new net N$13: R5.1
- new net N$14: R6.1
- new net N$15: R7.1
- new net N$16: R8.1
- new net N$17: Q1.B, R13.2
- new net N$18: Q1.C, R12.1, U12.P$2
- new net N$19: MS1.GPIOTX, R14.1
- new net N$2: R7.2, U7.1
- new net N$20: MS1.GPIORX, R15.1
- new net N$21: R14.2
- new net N$23: R15.2
- new net N$25: D1.C, U1.5
- new net N$26: D2.C, U2.5
- new net N$27: D3.C, U3.5
- new net N$28: D4.C, U4.5
- new net N$29: D5.C, U5.5
- new net N$3: R6.2, U6.1
- new net N$30: D6.C, U6.5
- new net N$31: D7.C, U7.5
- new net N$32: D8.C, U8.5
- new net N$4: R5.2, U5.1
- new net N$5: R4.2, U4.1
- new net N$6: R3.2, U3.1
- new net N$7: R2.2, U2.1
- new net N$8: R1.2, U1.1
- new net N$9: R1.1
- new net USB: D9.C, MS1.USB
- new net V_EXT1: U1.4, U1.6, U2.4, U2.6, U3.4, U3.6, U4.4, U4.6
- new net V_EXT2: U5.4, U5.6, U6.4, U6.6, U7.4, U7.6, U8.4, U8.6

Commit message: update
Parts:
- removed C1: (no value), GFE:C0603(1608)_HAND
- added JP1, JP2, JP3, JP4: JP2, GFE:JP2
- added R16, R17, R18, R19: 4.7k, GFE:R0603(1608)_HAND
Connections:
- removed net N$10: R2.1
- removed net N$11: R3.1
- removed net N$12: R4.1
- removed net N$13: R5.1
- removed net N$14: R6.1
- removed net N$15: R7.1
- removed net N$16: R8.1
- removed net N$21: R14.2
- removed net N$23: R15.2
- removed net N$9: R1.1
- new net 10: JP1.2, MS1.GPIO10
- new net 12: JP2.2, MS1.GPIO12
- new net GPS_PPS: JP3.1, R19.1
- new net GPS_RX: R14.2, U11.RX
- new net GPS_TX: R15.2, U11.TX
- new net HP_OUT: MS1.GPIO6
- new net MISO: R16.2, U10.SDO, U9.SDO
- new net MOSI: R17.2, U10.SDI, U9.SDI
- new net N$22: MS1.GPIOMISO, R16.1
- new net N$24: MS1.GPIOMOSI, R17.1
- new net N$33: MS1.GPIOSCK, R18.1
- new net N$34: R19.2, U11.PPS
- new net OUT_A1: MS1.GPIOA0, R8.1
- new net OUT_A2: MS1.GPIOA1, R7.1
- new net OUT_A3: MS1.GPIOA2, R6.1
- new net OUT_A4: MS1.GPIOA3, R5.1
- new net OUT_B1: MS1.GPIOA4, R4.1
- new net OUT_B2: MS1.GPIOA5, R3.1
- new net OUT_B3: JP4.1, R2.1
- new net OUT_B4: MS1.GPIO5, R1.1
- new net SCK: R18.2, U10.SCK, U9.SCK
- new net SCL: JP4.2, MS1.GPIOSCL
- new net SCL_EXT: JP4.3
- new net SDA: JP3.2, MS1.GPIOSDA
- new net SDA_EXT: JP3.3
- new net SERVO_1: MS1.GPIO9
- new net SERVO_2: JP1.3
- new net SERVO_3: JP2.3
- new net TEMP1_CS: JP1.1, U9.CS
- new net TEMP2_CS: JP2.1, U10.CS
- net +3V3: now also U10.VIN, U11.VIN, U9.VIN
- net BUZZER: now also MS1.GPIO11
- net GND: now also U10.GND, U11.GND, U9.GND
Other:
- moved on the sheet: D9, R14, R15

Commit message: update
Connections:
- new net N$10: R10.2
- new net N$11: R11.2
- new net N$9: R9.2
- net SERVO_1: now also R9.1
- net SERVO_2: now also R10.1
- net SERVO_3: now also R11.1
Other:
- moved on the sheet: R10, R11, R12, R19, R9, U10, U11, U9

Commit message: update
Parts:
- added D10: MBR120, GFE:MBR120
- added H1, H2, H3, H4: MOUNT-HOLE4.1, holes:MOUNT-HOLE4.1
- added Q2: NVF6P02, GFE:NVF6P02
- added S1: (no value), GFE:SWITCH
- added X1, X2, X3: 5267-03, GFE:5267-03
- added X10, X11, X12, X13, X14, X4, X5, X6, X7, X8, X9: 5267-02, GFE:5267-02
Connections:
- removed net USB: D9.C, MS1.USB
- new net EXT_5V: Q2.D, X4.1
- new net LED1: MS1.GPIO13
- net +5V: now also Q2.S, X1.1, X2.1, X3.1; no longer D9.A
- net GND: now also Q2.G, X1.3, X2.3, X3.3, X4.2
- net GND_EXT1: now also X10.2, X5.2, X7.2, X8.2, X9.2
- net GND_EXT2: now also X11.2, X12.2, X13.2, X14.2, X6.2
- net N$10: now also X2.2
- net N$11: now also X3.2
- net N$25: now also X7.1
- net N$26: now also X8.1
- net N$27: now also X9.1
- net N$28: now also X10.1
- net N$29: now also X11.1
- net N$30: now also X12.1
- net N$31: now also X13.1
- net N$32: now also X14.1
- net N$9: now also X1.2
- net V_EXT1: now also X5.1
- net V_EXT2: now also X6.1
Other:
- note added: "TODO: USB <-> 5V collison!"
- note added: "TODO: capacitor for servo!"
- moved on the sheet: D9, R10, R11, R9

Commit message: layout almost done
Parts:
- removed D10: MBR120, GFE:MBR120
- removed H3: MOUNT-HOLE4.1, holes:MOUNT-HOLE4.1
- removed S1: (no value), GFE:SWITCH
- added C1: (no value), adafruit:CPOL-USE3.5-8
- added JP5, JP6: M02PTH, berry:M02PTH
- added LOGO1: GRADEFREELOGO-20, GFE:GRADEFREELOGO-20
- added Q4: BC817-16LT1SMD, GFE:BC817-16LT1SMD
- added R22, R23: 1k, GFE:R0603(1608)_HAND
- added U13: NL17SZ17, GFE:NL17SZ17
- added X15: 5267-02, GFE:5267-02
- D1, D2, D3, D4, D5, D6, D7, D8: device GFE:MBR5200VPTR-E1 -> GFE:MBR5200VPTR-E1_V
- R10, R11, R9: value 4.7k -> 390
Connections:
- new net HP_SSR: U13.P$4, X15.1
- new net N$13: JP5.2, R23.2
- new net N$14: Q4.C, R23.1
- new net N$15: Q4.B, R22.2
- new net USB: D9.C, JP6.2, MS1.USB
- net +5V: now also C1.+, D9.A, JP5.1, JP6.1, U13.P$5
- net GND: now also C1.-, Q4.E, U13.P$3, X15.2
- net HP_OUT: now also U13.P$2
- net LED1: now also R22.1
Other:
- note added: "5V reverse voltage protection"
- note added: "TODO: solve USB power back-feeding!!"
- note removed: "TODO: USB <-> 5V collison!"
- moved on the sheet: D9

Commit message: updated
Parts:
- removed JP6: M02PTH, berry:M02PTH
- added J1: (no value), SparkFun-Connectors:CONN_04
- added LED1: (no value), GFE:LED3MM
- added R20: 500, GFE:R0603(1608)_HAND
- added X16: USB+SHIELD, GFE:USB+SHIELD
Connections:
- removed net USB: D9.C, JP6.2, MS1.USB
- new net D+: J1.3, X16.D+
- new net D-: J1.2, X16.D-
- new net N$12: D9.A, X16.VBUS
- new net N$16: LED1.A, R20.1
- new net STRUT_GND: X16.S1, X16.S2
- new net VBUS: D9.C, J1.1
- net +5V: now also MS1.USB, R20.2; no longer D9.A, JP6.1
- net GND: now also J1.4, LED1.C, X16.GND
Other:
- moved on the sheet: D9
Changed lines of the file:
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@@
 <layer number="112" name="tSilk" color="7" fill="1" visible="no" active="yes"/>
 <layer number="113" name="ReferenceLS" color="7" fill="1" visible="no" active="no"/>
+<layer number="114" name="Badge_Outline" color="7" fill="1" visible="yes" active="yes"/>
+<layer number="115" name="ReferenceISLANDS" color="7" fill="1" visible="yes" active="yes"/>
 <layer number="116" name="Patch_BOT" color="9" fill="4" visible="no" active="yes"/>
 <layer number="118" name="Rect_Pads" color="7" fill="1" visible="no" active="no"/>
@@
 <part name="C1" library="adafruit" deviceset="CPOL-US" device="E3.5-8"/>
 <part name="D9" library="GFE" deviceset="MBR120" device=""/>
-<part name="JP6" library="berry" deviceset="M02" device="PTH"/>
 <part name="LOGO1" library="GFE" deviceset="GRADEFREELOGO" device="-20"/>
+<part name="LED1" library="GFE" deviceset="LED" device="3MM"/>
+<part name="X16" library="GFE" deviceset="USB+SHIELD" device=""/>
+<part name="GND17" library="GFE" deviceset="GND" device=""/>
+<part name="J1" library="SparkFun-Connectors" deviceset="CONN_04" device=""/>
+<part name="GND24" library="GFE" deviceset="GND" device=""/>
+<part name="STRUT_GND1" library="GFE" deviceset="STRUT_GND" device=""/>
+<part name="R20" library="GFE" deviceset="R" device="0603(1608)_HAND" value="500"/>
+<part name="GND25" library="GFE" deviceset="GND" device=""/>
+<part name="P+6" library="supply1" deviceset="+5V" device=""/>
 </parts>
 <sheets>
 <sheet>
 <plain>
-<text x="220.98" y="226.06" size="1.778" layer="91">TODO: capacitor for servo!</text>
+<text x="182.88" y="210.82" size="1.778" layer="91">TODO: capacitor for servo!</text>
 <text x="172.72" y="213.36" size="1.778" layer="91">5V reverse voltage protection</text>
 <text x="53.34" y="88.9" size="1.778" layer="91">TODO: solve USB power back-feeding!!</text>
@@
 <instance part="U8" gate="G$1" x="236.22" y="83.82"/>
 <instance part="+3V1" gate="G$1" x="139.7" y="104.14" rot="R270"/>
-<instance part="P+1" gate="1" x="63.5" y="116.84" rot="R90"/>
+<instance part="P+1" gate="1" x="71.12" y="116.84" rot="R90"/>
 <instance part="V_EXT1" gate="1" x="246.38" y="213.36"/>
 <instance part="V_EXT2" gate="G$1" x="246.38" y="139.7"/>
@@
 <instance part="JP5" gate="G$1" x="195.58" y="60.96" rot="R180"/>
 <instance part="C1" gate="G$1" x="208.28" y="228.6" rot="MR0"/>
-<instance part="D9" gate="G$1" x="76.2" y="116.84"/>
-<instance part="JP6" gate="G$1" x="76.2" y="101.6" rot="MR90"/>
+<instance part="D9" gate="G$1" x="73.66" y="63.5" rot="R180"/>
 <instance part="LOGO1" gate="G$1" x="335.28" y="66.04"/>
+<instance part="LED1" gate="G$1" x="220.98" y="231.14"/>
+<instance part="X16" gate="G$1" x="88.9" y="60.96"/>
+<instance part="GND17" gate="1" x="83.82" y="55.88"/>
+<instance part="J1" gate="G$1" x="78.74" y="38.1"/>
+<instance part="GND24" gate="1" x="91.44" y="43.18" rot="R90"/>
+<instance part="STRUT_GND1" gate="G$1" x="91.44" y="50.8"/>
+<instance part="R20" gate="G$1" x="220.98" y="241.3" rot="R90"/>
+<instance part="GND25" gate="1" x="220.98" y="220.98"/>
+<instance part="P+6" gate="1" x="220.98" y="251.46"/>
 </instances>
 <busses>
@@
 <pinref part="Q4" gate="G$1" pin="E"/>
 <wire x1="182.88" y1="27.94" x2="182.88" y2="30.48" width="0.1524" layer="91"/>
+</segment>
+<segment>
+<pinref part="X16" gate="G$1" pin="GND"/>
+<pinref part="GND17" gate="1" pin="GND"/>
+<wire x1="86.36" y1="60.96" x2="83.82" y2="60.96" width="0.1524" layer="91"/>
+<wire x1="83.82" y1="60.96" x2="83.82" y2="58.42" width="0.1524" layer="91"/>
+</segment>
+<segment>
+<pinref part="GND24" gate="1" pin="GND"/>
+<pinref part="J1" gate="G$1" pin="4"/>
+<wire x1="88.9" y1="43.18" x2="83.82" y2="43.18" width="0.1524" layer="91"/>
+</segment>
+<segment>
+<pinref part="LED1" gate="G$1" pin="C"/>
+<pinref part="GND25" gate="1" pin="GND"/>
+<wire x1="220.98" y1="223.52" x2="220.98" y2="226.06" width="0.1524" layer="91"/>
 </segment>
 </net>
@@
 </segment>
 <segment>
+<pinref part="R20" gate="G$1" pin="2"/>
+<pinref part="P+6" gate="1" pin="+5V"/>
+<wire x1="220.98" y1="248.92" x2="220.98" y2="246.38" width="0.1524" layer="91"/>
+</segment>
+<segment>
 <pinref part="P+1" gate="1" pin="+5V"/>
-<pinref part="D9" gate="G$1" pin="A"/>
-<wire x1="66.04" y1="116.84" x2="71.12" y2="116.84" width="0.1524" layer="91"/>
-<wire x1="71.12" y1="116.84" x2="73.66" y2="116.84" width="0.1524" layer="91"/>
-<wire x1="76.2" y1="109.22" x2="71.12" y2="109.22" width="0.1524" layer="91"/>
-<wire x1="71.12" y1="109.22" x2="71.12" y2="116.84" width="0.1524" layer="91"/>
-<junction x="71.12" y="116.84"/>
-<pinref part="JP6" gate="G$1" pin="1"/>
+<pinref part="MS1" gate="G$1" pin="USB"/>
+<wire x1="73.66" y1="116.84" x2="91.44" y2="116.84" width="0.1524" layer="91"/>
 </segment>
 </net>
@@
 </segment>
 </net>
-<net name="USB" class="0">
-<segment>
-<pinref part="MS1" gate="G$1" pin="USB"/>
-<label x="88.9" y="116.84" size="1.778" layer="95" rot="R180" xref="yes"/>
-<pinref part="D9" gate="G$1" pin="C"/>
-<wire x1="78.74" y1="116.84" x2="83.82" y2="116.84" width="0.1524" layer="91"/>
-<wire x1="83.82" y1="116.84" x2="91.44" y2="116.84" width="0.1524" layer="91"/>
-<wire x1="78.74" y1="109.22" x2="83.82" y2="109.22" width="0.1524" layer="91"/>
-<wire x1="83.82" y1="109.22" x2="83.82" y2="116.84" width="0.1524" layer="91"/>
-<junction x="83.82" y="116.84"/>
-<pinref part="JP6" gate="G$1" pin="2"/>
-</segment>
-</net>
 <net name="HP_SSR" class="0">
 <segment>
@@
 </segment>
 </net>
+<net name="VBUS" class="0">
+<segment>
+<pinref part="J1" gate="G$1" pin="1"/>
+<wire x1="83.82" y1="35.56" x2="88.9" y2="35.56" width="0.1524" layer="91"/>
+<label x="88.9" y="35.56" size="1.778" layer="95" xref="yes"/>
+</segment>
+<segment>
+<pinref part="D9" gate="G$1" pin="C"/>
+<wire x1="71.12" y1="63.5" x2="66.04" y2="63.5" width="0.1524" layer="91"/>
+<label x="66.04" y="63.5" size="1.778" layer="95" rot="R180" xref="yes"/>
+</segment>
+</net>
+<net name="D-" class="0">
+<segment>
+<pinref part="X16" gate="G$1" pin="D-"/>
+<wire x1="86.36" y1="66.04" x2="81.28" y2="66.04" width="0.1524" layer="91"/>
+<label x="81.28" y="66.04" size="1.778" layer="95" rot="R180" xref="yes"/>
+</segment>
+<segment>
+<pinref part="J1" gate="G$1" pin="2"/>
+<wire x1="83.82" y1="38.1" x2="88.9" y2="38.1" width="0.1524" layer="91"/>
+<label x="88.9" y="38.1" size="1.778" layer="95" xref="yes"/>
+</segment>
+</net>
+<net name="D+" class="0">
+<segment>
+<pinref part="X16" gate="G$1" pin="D+"/>
+<wire x1="86.36" y1="68.58" x2="81.28" y2="68.58" width="0.1524" layer="91"/>
+<label x="81.28" y="68.58" size="1.778" layer="95" rot="R180" xref="yes"/>
+</segment>
+<segment>
+<pinref part="J1" gate="G$1" pin="3"/>
+<wire x1="83.82" y1="40.64" x2="88.9" y2="40.64" width="0.1524" layer="91"/>
+<label x="88.9" y="40.64" size="1.778" layer="95" xref="yes"/>
+</segment>
+</net>
+<net name="N$12" class="0">
+<segment>
+<pinref part="X16" gate="G$1" pin="VBUS"/>
+<pinref part="D9" gate="G$1" pin="A"/>
+<wire x1="86.36" y1="63.5" x2="76.2" y2="63.5" width="0.1524" layer="91"/>
+</segment>
+</net>
+<net name="STRUT_GND" class="0">
+<segment>
+<pinref part="STRUT_GND1" gate="G$1" pin="STRUT_GND"/>
+<pinref part="X16" gate="G$1" pin="S1"/>
+<wire x1="91.44" y1="50.8" x2="91.44" y2="53.34" width="0.1524" layer="91"/>
+<pinref part="X16" gate="G$1" pin="S2"/>
+<wire x1="91.44" y1="53.34" x2="91.44" y2="55.88" width="0.1524" layer="91"/>
+<wire x1="91.44" y1="53.34" x2="93.98" y2="53.34" width="0.1524" layer="91"/>
+<wire x1="93.98" y1="53.34" x2="93.98" y2="55.88" width="0.1524" layer="91"/>
+<junction x="91.44" y="53.34"/>
+</segment>
+</net>
+<net name="N$16" class="0">
+<segment>
+<pinref part="LED1" gate="G$1" pin="A"/>
+<pinref part="R20" gate="G$1" pin="1"/>
+<wire x1="220.98" y1="233.68" x2="220.98" y2="236.22" width="0.1524" layer="91"/>
+</segment>
+</net>

Commit message: tired
Parts:
- removed Q4: BC817-16LT1SMD, GFE:BC817-16LT1SMD
- removed R23: 1k, GFE:R0603(1608)_HAND
- added H3: MOUNT-HOLE4.1, holes:MOUNT-HOLE4.1
- added Q3: NVF6P02, GFE:NVF6P02
- added R21: 390, GFE:R0603(1608)_HAND
- C1: value (none) -> 0.1uF; device adafruit:CPOL-USE3.5-8 -> GFE:C0603(1608)_HAND
- C2: value 0.1uF -> (none); device GFE:C0603(1608)_HAND -> adafruit:CPOL-USE3.5-8
- D1: value (none) -> MBR120; device GFE:MBR5200VPTR-E1_V -> GFE:MBR120
- D9: value MBR120 -> (none); device GFE:MBR120 -> GFE:MBR5200VPTR-E1_V
- Q2: value NVF6P02 -> BC817-16LT1SMD; device GFE:NVF6P02 -> GFE:BC817-16LT1SMD
- R10, R11, R4, R7, R8, R9: value 390 -> 4.7k
- R14: value 4.7k -> 500
- R15, R16, R17, R18, R19: value 4.7k -> 390
- R20: value 500 -> 390
- R22: value 1k -> 390
- R5, R6: value 390 -> 1k
- U1, U2: value PVN012PBF -> MAX31856_ADAFRUIT; device GFE:PVN012PBF -> GFE:MAX31856_ADAFRUIT
- U10, U9: value MAX31856_ADAFRUIT -> PVN012PBF; device GFE:MAX31856_ADAFRUIT -> GFE:PVN012PBF
- U11: value GPS_ADAFRUIT -> PVN012PBF; device GFE:GPS_ADAFRUIT -> GFE:PVN012PBF
- U12: value BUZZER -> PVN012PBF; device GFE:BUZZER -> GFE:PVN012PBF
- U13: value NL17SZ17 -> PVN012PBF; device GFE:NL17SZ17 -> GFE:PVN012PBF
- U3: value PVN012PBF -> NL17SZ17; device GFE:PVN012PBF -> GFE:NL17SZ17
- U4: value PVN012PBF -> GPS_ADAFRUIT; device GFE:PVN012PBF -> GFE:GPS_ADAFRUIT
- U5: value PVN012PBF -> BUZZER; device GFE:PVN012PBF -> GFE:BUZZER
- X16: value USB+SHIELD -> 5267-02; device GFE:USB+SHIELD -> GFE:5267-02
- X4: value 5267-02 -> USB+SHIELD; device GFE:5267-02 -> GFE:USB+SHIELD
Connections:
- net +3V3: now also U1.VIN, U2.VIN, U4.VIN; no longer U10.VIN, U11.VIN, U9.VIN
- net +5V: now also C1.1, C2.+, Q3.S, R14.2, R6.2, U3.P$5, U5.P$1; no longer C1.+, C2.1, Q2.S, R12.2, R20.2, U12.P$1, U13.P$5
- net 10: now also JP3.2; no longer JP1.2
- net 12: now also JP4.2; no longer JP2.2
- net BUZZER: now also R5.1; no longer R13.1
- net D+: now also X4.D+; no longer X16.D+
- net D-: now also X4.D-; no longer X16.D-
- net EXT_5V: now also Q3.D, X6.1; no longer Q2.D, X4.1
- net GND: now also C1.2, C2.-, Q2.E, Q3.G, U1.GND, U10.2, U11.2, U12.2, U13.2, U2.GND, U3.P$3, U4.GND, U9.2, X4.GND, X5.2, X6.2; no longer C1.-, C2.2, Q2.G, Q4.E, U1.2, U10.GND, U11.GND, U13.P$3, U2.2, U3.2, U4.2, U5.2, U9.GND, X15.2, X16.GND, X4.2
- net GND_EXT1: now also D5.A, X11.2; no longer D1.A, X5.2
- net GND_EXT2: now also D9.A, X15.2, X16.2; no longer D5.A, X11.2, X6.2
- net GPS_PPS: now also JP1.1, R4.1; no longer JP3.1, R19.1
- net GPS_RX: now also R7.2, U4.RX; no longer R14.2, U11.RX
- net GPS_TX: now also R8.2, U4.TX; no longer R15.2, U11.TX
- net HP_OUT: now also U3.P$2; no longer U13.P$2
- net HP_SSR: now also U3.P$4, X5.1; no longer U13.P$4, X15.1
- net LED1: now also R12.1; no longer R22.1
- net MISO: now also R9.2, U1.SDO, U2.SDO; no longer R16.2, U10.SDO, U9.SDO
- net MOSI: now also R10.2, U1.SDI, U2.SDI; no longer R17.2, U10.SDI, U9.SDI
- net N$1: now also R22.2, U13.1; no longer R8.2, U8.1
- net N$10: now also R2.2; no longer R10.2
- net N$11: now also R3.2; no longer R11.2
- net N$12: now also D1.A, X4.VBUS; no longer D9.A, X16.VBUS
- net N$13: now also R13.2; no longer R23.2
- net N$14: now also Q2.C, R13.1; no longer Q4.C, R23.1
- net N$15: now also Q2.B, R12.2; no longer Q4.B, R22.2
- net N$16: now also R14.1; no longer R20.1
- net N$17: now also R5.2; no longer R13.2
- net N$18: now also R6.1, U5.P$2; no longer R12.1, U12.P$2
- net N$19: now also R7.1; no longer R14.1
- net N$2: now also R21.2, U12.1; no longer R7.2, U7.1
- net N$20: now also R8.1; no longer R15.1
- net N$22: now also R9.1; no longer R16.1
- net N$24: now also R10.1; no longer R17.1
- net N$25: now also D2.C, U6.5, X8.1; no longer D1.C, U1.5, X7.1
- net N$26: now also D3.C, U7.5, X9.1; no longer D2.C, U2.5, X8.1
- net N$27: now also D4.C, U8.5, X10.1; no longer D3.C, U3.5, X9.1
- net N$28: now also D5.C, U9.5, X11.1; no longer D4.C, U4.5, X10.1
- net N$29: now also D6.C, U10.5, X12.1; no longer D5.C, U5.5, X11.1
- net N$3: now also R20.2, U11.1; no longer R6.2, U6.1
- net N$30: now also D7.C, U11.5, X13.1; no longer D6.C, U6.5, X12.1
- net N$31: now also D8.C, U12.5, X14.1; no longer D7.C, U7.5, X13.1
- net N$32: now also D9.C, U13.5, X15.1; no longer D8.C, U8.5, X14.1
- net N$33: now also R11.1; no longer R18.1
- net N$34: now also R4.2, U4.PPS; no longer R19.2, U11.PPS
- net N$4: now also R19.2, U10.1; no longer R5.2, U5.1
- net N$5: now also R18.2, U9.1; no longer R4.2, U4.1
- net N$6: now also R17.2, U8.1; no longer R3.2, U3.1
- net N$7: now also R16.2, U7.1; no longer R2.2, U2.1
- net N$8: now also R15.2, U6.1; no longer R1.2, U1.1
- net N$9: now also R1.2; no longer R9.2
- net OUT_A1: now also R22.1; no longer R8.1
- net OUT_A2: now also R21.1; no longer R7.1
- net OUT_A3: now also R20.1; no longer R6.1
- net OUT_A4: now also R19.1; no longer R5.1
- net OUT_B1: now also R18.1; no longer R4.1
- net OUT_B2: now also R17.1; no longer R3.1
- net OUT_B3: now also JP2.1, R16.1; no longer JP4.1, R2.1
- net OUT_B4: now also R15.1; no longer R1.1
- net SCK: now also R11.2, U1.SCK, U2.SCK; no longer R18.2, U10.SCK, U9.SCK
- net SCL: now also JP2.2; no longer JP4.2
- net SCL_EXT: now also JP2.3; no longer JP4.3
- net SDA: now also JP1.2; no longer JP3.2
- net SDA_EXT: now also JP1.3; no longer JP3.3
- net SERVO_1: now also R1.1; no longer R9.1
- net SERVO_2: now also JP3.3, R2.1; no longer JP1.3, R10.1
- net SERVO_3: now also JP4.3, R3.1; no longer JP2.3, R11.1
- net STRUT_GND: now also X4.S1, X4.S2; no longer X16.S1, X16.S2
- net TEMP1_CS: now also JP3.1, U1.CS; no longer JP1.1, U9.CS
- net TEMP2_CS: now also JP4.1, U2.CS; no longer JP2.1, U10.CS
- net VBUS: now also D1.C; no longer D9.C
- net V_EXT1: now also U6.4, U6.6, U7.4, U7.6, U8.4, U8.6, U9.4, U9.6, X7.1; no longer U1.4, U1.6, U2.4, U2.6, U3.4, U3.6, U4.4, U4.6, X5.1
- net V_EXT2: now also U10.4, U10.6, U11.4, U11.6, U12.4, U12.6, U13.4, U13.6, X16.1; no longer U5.4, U5.6, U6.4, U6.6, U7.4, U7.6, U8.4, U8.6, X6.1
Other:
- moved on the sheet: D1, D2, D3, D4, D5, D6, D7, D8, D9, H4, JP1, JP2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
