File: Ramyun/RamyunActionBoard.sch (EAGLE design)
At the start: 78 parts, among them Q1 BC817-16LT1SMD, Q2 BC817-16LT1SMD, Q3 NVF6P02, U1 MAX31856_ADAFRUIT, U10 PVN012PBF, U11 PVN012PBF, U12 PVN012PBF, U13 PVN012PBF, U2 MAX31856_ADAFRUIT, U3 NL17SZ17, U4 GPS_ADAFRUIT, U5 BUZZER, U6 PVN012PBF, U7 PVN012PBF, U8 PVN012PBF, U9 PVN012PBF, X1 5267-03, X10 5267-02, X11 5267-02, X12 5267-02, X13 5267-02, X14 5267-02, X15 5267-02, X16 5267-02, X2 5267-03, X3 5267-03, X4 USB+SHIELD, X5 5267-02, X6 5267-02, X7 5267-02, X8 5267-02, X9 5267-02

Commit message: tired 2
Parts:
- added TP1, TP2, TP3, TP4, TP5, TP6: (no value), berry:TP-5010
Connections:
- net +5V: now also TP1.TP
- net GND: now also TP4.TP
- net GND_EXT1: now also TP5.TP
- net GND_EXT2: now also TP6.TP
- net V_EXT1: now also TP2.TP
- net V_EXT2: now also TP3.TP
Changed lines of the file:
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@@
 <part name="P+9" library="supply1" deviceset="+5V" device=""/>
 <part name="H4" library="holes" deviceset="MOUNT-HOLE" device="4.1"/>
+<part name="TP1" library="berry" deviceset="TP" device="-5010"/>
+<part name="TP2" library="berry" deviceset="TP" device="-5010"/>
+<part name="TP3" library="berry" deviceset="TP" device="-5010"/>
+<part name="TP4" library="berry" deviceset="TP" device="-5010"/>
+<part name="P+10" library="supply1" deviceset="+5V" device=""/>
+<part name="V_EXT1" library="GFE" deviceset="V_EXT1" device=""/>
+<part name="V_EXT2" library="GFE" deviceset="V_EXT2" device=""/>
+<part name="TP5" library="berry" deviceset="TP" device="-5010"/>
+<part name="GND26" library="GFE" deviceset="GND" device=""/>
+<part name="TP6" library="berry" deviceset="TP" device="-5010"/>
+<part name="GND_EXT1" library="GFE" deviceset="GND_EXT2" device=""/>
+<part name="GND_EXT2" library="GFE" deviceset="GND_EXT1" device=""/>
 </parts>
 <sheets>
@@
 <instance part="P+9" gate="1" x="220.98" y="251.46"/>
 <instance part="H4" gate="G$1" x="248.92" y="25.4"/>
+<instance part="TP1" gate="G$1" x="327.66" y="223.52"/>
+<instance part="TP2" gate="G$1" x="337.82" y="223.52"/>
+<instance part="TP3" gate="G$1" x="345.44" y="223.52"/>
+<instance part="TP4" gate="G$1" x="353.06" y="223.52"/>
+<instance part="P+10" gate="1" x="322.58" y="218.44" rot="R90"/>
+<instance part="V_EXT1" gate="1" x="332.74" y="218.44" rot="R90"/>
+<instance part="V_EXT2" gate="G$1" x="340.36" y="218.44" rot="R90"/>
+<instance part="TP5" gate="G$1" x="360.68" y="223.52"/>
+<instance part="GND26" gate="1" x="353.06" y="213.36"/>
+<instance part="TP6" gate="G$1" x="368.3" y="223.52"/>
+<instance part="GND_EXT1" gate="G$1" x="368.3" y="213.36"/>
+<instance part="GND_EXT2" gate="G$1" x="360.68" y="213.36"/>
 </instances>
 <busses>
@@
 <pinref part="GND16" gate="1" pin="GND"/>
 <wire x1="220.98" y1="223.52" x2="220.98" y2="226.06" width="0.1524" layer="91"/>
+</segment>
+<segment>
+<pinref part="GND26" gate="1" pin="GND"/>
+<pinref part="TP4" gate="G$1" pin="TP"/>
+<wire x1="353.06" y1="215.9" x2="353.06" y2="220.98" width="0.1524" layer="91"/>
 </segment>
 </net>
@@
 <pinref part="X7" gate="G$1" pin="2"/>
 </segment>
+<segment>
+<pinref part="TP5" gate="G$1" pin="TP"/>
+<wire x1="360.68" y1="215.9" x2="360.68" y2="220.98" width="0.1524" layer="91"/>
+<pinref part="GND_EXT2" gate="G$1" pin="GND_EXT1"/>
+</segment>
 </net>
 <net name="V_EXT1" class="0">
@@
 <wire x1="279.4" y1="243.84" x2="284.48" y2="243.84" width="0.1524" layer="91"/>
 <pinref part="X7" gate="G$1" pin="1"/>
+</segment>
+<segment>
+<pinref part="V_EXT1" gate="1" pin="V_EXT1"/>
+<pinref part="TP2" gate="G$1" pin="TP"/>
+<wire x1="335.28" y1="218.44" x2="337.82" y2="218.44" width="0.1524" layer="91"/>
+<wire x1="337.82" y1="218.44" x2="337.82" y2="220.98" width="0.1524" layer="91"/>
 </segment>
 </net>
@@
 <pinref part="X16" gate="G$1" pin="2"/>
 </segment>
+<segment>
+<pinref part="TP6" gate="G$1" pin="TP"/>
+<wire x1="368.3" y1="215.9" x2="368.3" y2="220.98" width="0.1524" layer="91"/>
+<pinref part="GND_EXT1" gate="G$1" pin="GND_EXT2"/>
+</segment>
 </net>
 <net name="V_EXT2" class="0">
@@
 <wire x1="304.8" y1="243.84" x2="309.88" y2="243.84" width="0.1524" layer="91"/>
 <pinref part="X16" gate="G$1" pin="1"/>
+</segment>
+<segment>
+<pinref part="V_EXT2" gate="G$1" pin="V_EXT2"/>
+<pinref part="TP3" gate="G$1" pin="TP"/>
+<wire x1="342.9" y1="218.44" x2="345.44" y2="218.44" width="0.1524" layer="91"/>
+<wire x1="345.44" y1="218.44" x2="345.44" y2="220.98" width="0.1524" layer="91"/>
 </segment>
 </net>
@@
 <wire x1="73.66" y1="116.84" x2="91.44" y2="116.84" width="0.1524" layer="91"/>
 </segment>
+<segment>
+<pinref part="P+10" gate="1" pin="+5V"/>
+<pinref part="TP1" gate="G$1" pin="TP"/>
+<wire x1="325.12" y1="218.44" x2="327.66" y2="218.44" width="0.1524" layer="91"/>
+<wire x1="327.66" y1="218.44" x2="327.66" y2="220.98" width="0.1524" layer="91"/>
+</segment>
 </net>
 <net name="N$19" class="0">
@@
 <segment>
 <pinref part="MS1" gate="G$1" pin="GPIOSDA"/>
-<wire x1="91.44" y1="139.7" x2="86.36" y2="139.7" width="0.1524" layer="91"/>
-<label x="86.36" y="139.7" size="1.778" layer="95" rot="R180" xref="yes"/>
+<wire x1="91.44" y1="139.7" x2="76.2" y2="139.7" width="0.1524" layer="91"/>
+<label x="76.2" y="139.7" size="1.778" layer="95" rot="R180" xref="yes"/>
 </segment>
 <segment>
@@
 <segment>
 <pinref part="MS1" gate="G$1" pin="GPIOSCL"/>
-<wire x1="91.44" y1="137.16" x2="86.36" y2="137.16" width="0.1524" layer="91"/>
-<label x="86.36" y="137.16" size="1.778" layer="95" rot="R180" xref="yes"/>
-</segment>
-<segment>
+<wire x1="91.44" y1="137.16" x2="76.2" y2="137.16" width="0.1524" layer="91"/>
+<label x="76.2" y="137.16" size="1.778" layer="95" rot="R180" xref="yes"/>
+</segment>
+<segment>
