File: Ramyun/RamyunControlBoard.brd (EAGLE design)
At the start: 135.2 x 135.2 mm, 7 parts, among them IC1 MCP23017SO, X1 5267-02, X2 5267-03

Commit message: tired
Parts:
- added C2: (no value), adafruit:E3,5-8
- added C3: 0.1uF, GFE:C0603(1608)_HANDSOLDER
- added H1, H2, H3, H4: MOUNT-HOLE4.1, holes:4,1
- added J1, J2: (no value), SparkFun-Connectors:2X8
- added JP1: M02PTH, berry:1X02
- added LED2: (no value), GFE:LED3MM
- added LOGO1: GRADEFREELOGO-20, GFE:GRADEFREELOGO-20
- added Q1: NVF6P02, GFE:SOT223
- added Q2: BC817-16LT1SMD, GFE:SOT23-BEC
- added R10, R11: 100k, GFE:R0603(1608)_HANDSOLDER
- added R12, R13, R14, R15, R16, R17, R18, R19, R2, R20, R3, R4, R5, R8: 4.7k, GFE:R0603(1608)_HANDSOLDER
- added R21, R39, R9: 500, GFE:R0603(1608)_HANDSOLDER
- added R22, R23, R24, R25, R26, R27, R28, R29, R30, R31, R32, R33, R34, R35, R36, R37: 470, GFE:R0603(1608)_HANDSOLDER
- added R38: 1k, GFE:R0603(1608)_HANDSOLDER
- added R6, R7: 390, GFE:R0603(1608)_HANDSOLDER
- added U1: LMP7702, GFE:DGK_S-DPSO-G8
- added X10, X11, X16, X3, X4, X5, X6, X7, X8, X9: 5267-02, GFE:5267-02
- added X12, X13, X14, X15, X17: 5267-03, GFE:5267-03
- C1: value (none) -> 0.1uF
- R1: value (none) -> 4.7k
- X2: value 5267-03 -> 5267-02; device GFE:5267-03 -> GFE:5267-02
- moved R1 180.3 mm to (52.1, 21.6), turned to 180 degrees
- moved C1 164.5 mm to (-20.3, 38.1), turned to 90 degrees
- moved LED1 131.0 mm to (16.5, -22.9), turned to 270 degrees
- moved X2 122.2 mm to (45.7, -40.6), turned to 90 degrees
- moved X1 103.4 mm to (33.0, -40.6), turned to 90 degrees
- moved IC1 78.3 mm to (-33.0, 0.00)
Connections:
- removed net VDD: IC1.9
- removed net VSS: IC1.10
- new net +5V: C2.+, Q1.3, R21.2, X12.1, X13.1
- new net ANALOG_1: MS1.5, U1.1, U1.2
- new net ANALOG_2: MS1.6, U1.6, U1.7
- new net BTN_1: R20.2, X1.1
- new net BTN_10: R3.1, X10.1
- new net BTN_11: R4.1, X11.1
- new net BTN_2: R19.2, X2.1
- new net BTN_3: R18.2, X3.1
- new net BTN_4: R17.2, X4.1
- new net BTN_5: R16.2, X5.1
- new net BTN_6: R15.2, X6.1
- new net BTN_7: R14.2, X7.1
- new net BTN_8: R1.1, X8.1
- new net BTN_9: R2.1, X9.1
- new net EXT_5V: Q1.2, Q1.4, X16.1
- new net IO_1: J2.15, R30.2
- new net IO_10: J1.13, R23.2
- new net IO_11: J1.11, R24.2
- new net IO_12: J1.9, R25.2
- new net IO_13: J1.7, R26.2
- new net IO_14: J1.5, R27.2
- new net IO_15: J1.3, R28.2
- new net IO_16: J1.1, R29.2
- new net IO_2: J2.13, R31.2
- new net IO_3: J2.11, R32.2
- new net IO_4: J2.9, R33.2
- new net IO_5: J2.7, R34.2
- new net IO_6: J2.5, R35.2
- new net IO_7: J2.3, R36.2
- new net IO_8: J2.1, R37.2
- new net IO_9: J1.15, R22.2
- new net LED_1: MS1.25, R38.1
- new net N$1: MS1.7, R20.1
- new net N$10: MS1.20, R2.2
- new net N$11: MS1.21, R3.2
- new net N$12: MS1.22, R4.2
- new net N$13: MS1.15, R12.1
- new net N$14: MS1.14, R13.1
- new net N$15: MS1.11, R16.1
- new net N$16: MS1.12, R15.1
- new net N$17: MS1.13, R14.1
- new net N$18: IC1.21, R30.1
- new net N$19: IC1.22, R31.1
- new net N$2: R10.2, U1.3
- new net N$20: IC1.23, R32.1
- new net N$21: IC1.24, R33.1
- new net N$22: IC1.25, R34.1
- new net N$23: IC1.26, R35.1
- new net N$24: IC1.27, R36.1
- new net N$25: IC1.28, R37.1
- new net N$26: IC1.1, R22.1
- new net N$27: IC1.2, R23.1
- new net N$28: IC1.3, R24.1
- new net N$29: IC1.4, R25.1
- new net N$3: R11.2, U1.5
- new net N$30: IC1.5, R26.1
- new net N$31: IC1.6, R27.1
- new net N$32: IC1.7, R28.1
- new net N$33: IC1.8, R29.1
- new net N$34: R6.1, X12.2
- new net N$35: R7.1, X13.2
- new net N$36: LED2.A, R21.1
- new net N$4: MS1.8, R19.1
- new net N$5: MS1.9, R18.1
- new net N$50: Q2.C, R39.1
- new net N$51: Q2.B, R38.2
- new net N$52: JP1.2, R39.2
- new net N$53: LED1.A, R9.1
- new net N$6: MS1.10, R17.1
- new net N$7: R11.1, X15.2
- new net N$8: R10.1, X14.2
- new net N$9: MS1.19, R1.2
- new net RXD: R13.2, X17.3
- new net SCL: IC1.12, MS1.18, R8.1
- new net SDA: IC1.13, MS1.17, R5.1
- new net SERVO_1: MS1.23, R6.2
- new net SERVO_2: MS1.24, R7.2
- new net TXD: R12.2, X17.2
- net 3.3V: now also C1.1, C3.1, IC1.18, IC1.9, R5.2, R8.2, R9.2, U1.8, X14.1, X15.1
- net GND: now also C1.2, C2.-, C3.2, IC1.10, IC1.15, IC1.16, IC1.17, J1.10, J1.12, J1.14, J1.16, J1.2, J1.4, J1.6, J1.8, J2.10, J2.12, J2.14, J2.16, J2.2, J2.4, J2.6, J2.8, LED1.K, LED2.K, Q1.1, Q2.E, U1.4, X1.2, X10.2, X11.2, X12.3, X13.3, X14.3, X15.3, X16.2, X17.1, X2.2, X3.2, X4.2, X5.2, X6.2, X7.2, X8.2, X9.2
- net VBUS: now also JP1.1
Other:
- board text added: "Project R"

Commit message: tired 2
Parts:
- added TP1, TP2: (no value), berry:TP-5010
Connections:
- net +5V: now also TP1.TP
- net GND: now also TP2.TP
Changed lines of the file:
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@@
 <layer number="17" name="Pads" color="2" fill="1" visible="yes" active="yes"/>
 <layer number="18" name="Vias" color="2" fill="1" visible="yes" active="yes"/>
-<layer number="19" name="Unrouted" color="6" fill="1" visible="no" active="yes"/>
+<layer number="19" name="Unrouted" color="6" fill="1" visible="yes" active="yes"/>
 <layer number="20" name="Dimension" color="15" fill="1" visible="yes" active="yes"/>
 <layer number="21" name="tPlace" color="7" fill="1" visible="yes" active="yes"/>
@@
 <element name="H3" library="holes" package="4,1" value="MOUNT-HOLE4.1" x="-60" y="0"/>
 <element name="H4" library="holes" package="4,1" value="MOUNT-HOLE4.1" x="30" y="0"/>
+<element name="TP1" library="berry" package="TP-5010" value="" x="-33.02" y="-36.83"/>
+<element name="TP2" library="berry" package="TP-5010" value="" x="-21.59" y="-36.83"/>
 </elements>
 <signals>
@@
 <contactref element="J1" pad="14"/>
 <contactref element="J1" pad="16"/>
-<wire x1="52.07" y1="29.23" x2="45.72" y2="39.39" width="0" layer="19" extent="1-1"/>
-<wire x1="57.15" y1="19.07" x2="52.07" y2="29.23" width="0" layer="19" extent="1-1"/>
-<wire x1="60.96" y1="8.91" x2="57.15" y2="19.07" width="0" layer="19" extent="1-1"/>
-<wire x1="60.96" y1="-1.25" x2="60.96" y2="8.91" width="0" layer="19" extent="1-1"/>
-<wire x1="60.96" y1="-11.41" x2="60.96" y2="-1.25" width="0" layer="19" extent="1-1"/>
-<wire x1="57.15" y1="-21.57" x2="60.96" y2="-11.41" width="0" layer="19" extent="1-1"/>
-<wire x1="52.07" y1="-31.73" x2="57.15" y2="-21.57" width="0" layer="19" extent="1-1"/>
-<wire x1="45.72" y1="-41.89" x2="52.07" y2="-31.73" width="0" layer="19" extent="1-1"/>
-<wire x1="33.02" y1="39.39" x2="45.72" y2="39.39" width="0" layer="19" extent="1-1"/>
-<wire x1="33.02" y1="-41.89" x2="45.72" y2="-41.89" width="0" layer="19" extent="1-1"/>
-<wire x1="22.86" y1="19.05" x2="33.02" y2="39.39" width="0" layer="19" extent="1-1"/>
-<wire x1="-23.81" y1="-25.57" x2="22.86" y2="19.05" width="0" layer="19" extent="1-1"/>
-<wire x1="-20.32" y1="39.25" x2="-23.81" y2="-25.57" width="0" layer="19" extent="1-1"/>
-<wire x1="-25.105" y1="40.3" x2="-20.32" y2="39.25" width="0" layer="19" extent="1-1"/>
-<wire x1="-33.02" y1="46.99" x2="-25.105" y2="40.3" width="0" layer="19" extent="1-1"/>
-<wire x1="-46.99" y1="34.29" x2="-33.02" y2="46.99" width="0" layer="19" extent="1-1"/>
-<wire x1="-57.15" y1="27.94" x2="-46.99" y2="34.29" width="0" layer="19" extent="1-1"/>
-<wire x1="-57.15" y1="25.4" x2="-57.15" y2="27.94" width="0" layer="19" extent="1-1"/>
-<wire x1="-57.15" y1="22.86" x2="-57.15" y2="25.4" width="0" layer="19" extent="1-1"/>
-<wire x1="-57.15" y1="20.32" x2="-57.15" y2="22.86" width="0" layer="19" extent="1-1"/>
-<wire x1="-57.15" y1="17.78" x2="-57.15" y2="20.32" width="0" layer="19" extent="1-1"/>
-<wire x1="-57.15" y1="15.24" x2="-57.15" y2="17.78" width="0" layer="19" extent="1-1"/>
-<wire x1="-57.15" y1="12.7" x2="-57.15" y2="15.24" width="0" layer="19" extent="1-1"/>
-<wire x1="-57.15" y1="10.16" x2="-57.15" y2="12.7" width="0" layer="19" extent="1-1"/>
-<wire x1="-57.15" y1="-10.16" x2="-57.15" y2="10.16" width="0" layer="19" extent="1-1"/>
-<wire x1="-57.15" y1="-12.7" x2="-57.15" y2="-10.16" width="0" layer="19" extent="1-1"/>
-<wire x1="-57.15" y1="-15.24" x2="-57.15" y2="-12.7" width="0" layer="19" extent="1-1"/>
-<wire x1="-57.15" y1="-17.78" x2="-57.15" y2="-15.24" width="0" layer="19" extent="1-1"/>
-<wire x1="-57.15" y1="-20.32" x2="-57.15" y2="-17.78" width="0" layer="19" extent="1-1"/>
-<wire x1="-57.15" y1="-22.86" x2="-57.15" y2="-20.32" width="0" layer="19" extent="1-1"/>
-<wire x1="-57.15" y1="-25.4" x2="-57.15" y2="-22.86" width="0" layer="19" extent="1-1"/>
-<wire x1="-57.15" y1="-27.94" x2="-57.15" y2="-25.4" width="0" layer="19" extent="1-1"/>
-<wire x1="-46.99" y1="-39.37" x2="-57.15" y2="-27.94" width="0" layer="19" extent="1-1"/>
-<wire x1="-33.02" y1="-52.07" x2="-46.99" y2="-39.37" width="0" layer="19" extent="1-1"/>
-<wire x1="-21.59" y1="-58.42" x2="-33.02" y2="-52.07" width="0" layer="19" extent="1-1"/>
+<contactref element="TP2" pad="TP"/>
+<wire x1="-21.59" y1="-58.42" x2="-21.59" y2="-36.83" width="0" layer="19" extent="1-1"/>
 <wire x1="-12.68" y1="-59.69" x2="-21.59" y2="-58.42" width="0" layer="19" extent="1-1"/>
 <wire x1="-9.13" y1="-48.92" x2="-12.68" y2="-59.69" width="0" layer="19" extent="1-1"/>
 <wire x1="-9.652" y1="-41.91" x2="-9.13" y2="-48.92" width="0" layer="19" extent="1-1"/>
-<wire x1="16.51" y1="-24.13" x2="-9.652" y2="-41.91" width="0" layer="19" extent="1-1"/>
-<wire x1="-29.21" y1="-4.78" x2="16.51" y2="-24.13" width="0" layer="19" extent="1-1"/>
+<wire x1="-33.02" y1="-52.07" x2="-21.59" y2="-58.42" width="0" layer="19" extent="1-1"/>
+<wire x1="-46.99" y1="-39.37" x2="-33.02" y2="-52.07" width="0" layer="19" extent="1-1"/>
+<wire x1="-57.15" y1="-27.94" x2="-46.99" y2="-39.37" width="0" layer="19" extent="1-1"/>
+<wire x1="-57.15" y1="-25.4" x2="-57.15" y2="-27.94" width="0" layer="19" extent="1-1"/>
+<wire x1="-57.15" y1="-22.86" x2="-57.15" y2="-25.4" width="0" layer="19" extent="1-1"/>
+<wire x1="-57.15" y1="-20.32" x2="-57.15" y2="-22.86" width="0" layer="19" extent="1-1"/>
+<wire x1="-57.15" y1="-17.78" x2="-57.15" y2="-20.32" width="0" layer="19" extent="1-1"/>
+<wire x1="-57.15" y1="-15.24" x2="-57.15" y2="-17.78" width="0" layer="19" extent="1-1"/>
+<wire x1="-57.15" y1="-12.7" x2="-57.15" y2="-15.24" width="0" layer="19" extent="1-1"/>
+<wire x1="-57.15" y1="-10.16" x2="-57.15" y2="-12.7" width="0" layer="19" extent="1-1"/>
+<wire x1="-57.15" y1="10.16" x2="-57.15" y2="-10.16" width="0" layer="19" extent="1-1"/>
+<wire x1="-57.15" y1="12.7" x2="-57.15" y2="10.16" width="0" layer="19" extent="1-1"/>
+<wire x1="-57.15" y1="15.24" x2="-57.15" y2="12.7" width="0" layer="19" extent="1-1"/>
+<wire x1="-57.15" y1="17.78" x2="-57.15" y2="15.24" width="0" layer="19" extent="1-1"/>
+<wire x1="-57.15" y1="20.32" x2="-57.15" y2="17.78" width="0" layer="19" extent="1-1"/>
+<wire x1="-57.15" y1="22.86" x2="-57.15" y2="20.32" width="0" layer="19" extent="1-1"/>
+<wire x1="-57.15" y1="25.4" x2="-57.15" y2="22.86" width="0" layer="19" extent="1-1"/>
+<wire x1="-57.15" y1="27.94" x2="-57.15" y2="25.4" width="0" layer="19" extent="1-1"/>
+<wire x1="-46.99" y1="34.29" x2="-57.15" y2="27.94" width="0" layer="19" extent="1-1"/>
+<wire x1="-33.02" y1="46.99" x2="-46.99" y2="34.29" width="0" layer="19" extent="1-1"/>
+<wire x1="-25.105" y1="40.3" x2="-33.02" y2="46.99" width="0" layer="19" extent="1-1"/>
+<wire x1="-20.32" y1="39.25" x2="-25.105" y2="40.3" width="0" layer="19" extent="1-1"/>
+<wire x1="-23.81" y1="-25.57" x2="-9.652" y2="-41.91" width="0" layer="19" extent="1-1"/>
+<wire x1="-29.21" y1="-4.78" x2="-23.81" y2="-25.57" width="0" layer="19" extent="1-1"/>
 <wire x1="-21.59" y1="1.15" x2="-29.21" y2="-4.78" width="0" layer="19" extent="1-1"/>
 <wire x1="-24.13" y1="4.78" x2="-21.59" y2="1.15" width="0" layer="19" extent="1-1"/>
 <wire x1="-25.4" y1="4.78" x2="-24.13" y2="4.78" width="0" layer="19" extent="1-1"/>
 <wire x1="-26.67" y1="4.78" x2="-25.4" y2="4.78" width="0" layer="19" extent="1-1"/>
-<wire x1="10.16" y1="-11.43" x2="22.86" y2="19.05" width="0" layer="19" extent="1-1"/>
+<wire x1="16.51" y1="-24.13" x2="-9.652" y2="-41.91" width="0" layer="19" extent="1-1"/>
+<wire x1="10.16" y1="-11.43" x2="16.51" y2="-24.13" width="0" layer="19" extent="1-1"/>
+<wire x1="33.02" y1="-41.89" x2="16.51" y2="-24.13" width="0" layer="19" extent="1-1"/>
+<wire x1="45.72" y1="-41.89" x2="33.02" y2="-41.89" width="0" layer="19" extent="1-1"/>
+<wire x1="52.07" y1="-31.73" x2="45.72" y2="-41.89" width="0" layer="19" extent="1-1"/>
+<wire x1="57.15" y1="-21.57" x2="52.07" y2="-31.73" width="0" layer="19" extent="1-1"/>
+<wire x1="60.96" y1="-11.41" x2="57.15" y2="-21.57" width="0" layer="19" extent="1-1"/>
+<wire x1="60.96" y1="-1.25" x2="60.96" y2="-11.41" width="0" layer="19" extent="1-1"/>
+<wire x1="60.96" y1="8.91" x2="60.96" y2="-1.25" width="0" layer="19" extent="1-1"/>
+<wire x1="57.15" y1="19.07" x2="60.96" y2="8.91" width="0" layer="19" extent="1-1"/>
+<wire x1="52.07" y1="29.23" x2="57.15" y2="19.07" width="0" layer="19" extent="1-1"/>
+<wire x1="45.72" y1="39.39" x2="52.07" y2="29.23" width="0" layer="19" extent="1-1"/>
+<wire x1="33.02" y1="39.39" x2="45.72" y2="39.39" width="0" layer="19" extent="1-1"/>
+<wire x1="22.86" y1="19.05" x2="33.02" y2="39.39" width="0" layer="19" extent="1-1"/>
 </signal>
 <signal name="VBUS">
@@
 <contactref element="X12" pad="1"/>
 <contactref element="X13" pad="1"/>
-<wire x1="-33.02" y1="-46.99" x2="-46.99" y2="-34.29" width="0" layer="19" extent="1-1"/>
+<contactref element="TP1" pad="TP"/>
+<wire x1="-33.02" y1="-46.99" x2="-33.02" y2="-36.83" width="0" layer="19" extent="1-1"/>
 <wire x1="-21.59" y1="-49.65" x2="-33.02" y2="-46.99" width="0" layer="19" extent="1-1"/>
 <wire x1="-13.73" y1="-48.92" x2="-21.59" y2="-49.65" width="0" layer="19" extent="1-1"/>
 <wire x1="-13.208" y1="-41.91" x2="-13.73" y2="-48.92" width="0" layer="19" extent="1-1"/>
+<wire x1="-46.99" y1="-34.29" x2="-33.02" y2="-46.99" width="0" layer="19" extent="1-1"/>
 </signal>
 <signal name="EXT_5V">

Commit message: gerber done
Parts:
- moved TP2 6.35 mm to (-27.9, -36.8)
- moved R15 2.54 mm to (55.9, -1.27)
- moved R1 2.54 mm to (52.1, 19.1)
- moved R14 2.54 mm to (55.9, 8.89)
- moved R16 2.54 mm to (55.9, -11.4)
- moved R17 2.54 mm to (52.1, -21.6)
- moved R18 2.54 mm to (47.0, -31.8)
- moved R19 2.54 mm to (40.6, -41.9)
- moved R2 2.54 mm to (47.0, 29.2)
- moved R20 2.54 mm to (27.9, -41.9)
- moved R11 1.27 mm to (-24.1, 31.8)
- moved X10 1.27 mm to (47.0, 40.6), turned to 270 degrees
- moved X2 1.27 mm to (47.0, -40.6), turned to 270 degrees
- moved X3 1.27 mm to (53.3, -30.5), turned to 270 degrees
- moved X4 1.27 mm to (58.4, -20.3), turned to 270 degrees
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Routing:
- net 3.3V: track 0.00 -> 161.0 mm, vias 0 -> 1
- net SERVO_2: track 0.00 -> 90.8 mm
- net N$10: track 0.00 -> 80.3 mm
- net N$9: track 0.00 -> 77.2 mm
- net ANALOG_1: track 0.00 -> 76.8 mm
- net N$11: track 0.00 -> 64.4 mm
- net ANALOG_2: track 0.00 -> 61.8 mm, vias 0 -> 1
- net +5V: track 0.00 -> 55.2 mm
- net SERVO_1: track 0.00 -> 52.9 mm, vias 0 -> 1
- net N$4: track 0.00 -> 52.7 mm
- net N$12: track 0.00 -> 52.4 mm
- net N$15: track 0.00 -> 51.9 mm
- net N$6: track 0.00 -> 51.3 mm
- net N$5: track 0.00 -> 49.4 mm
- net N$16: track 0.00 -> 49.2 mm
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- added copper zone on layer 16, net GND
Other:
- board text added: "5V"
- board text added: "AN 1"
- board text added: "AN 2"
- board text added: "BTN 1"
- board text added: "BTN 2"
- board text added: "BTN 3"
- board text added: "BTN 4"
- board text added: "BTN 5"
- board text added: "BTN 6"
- board text added: "BTN 7"
- board text added: "BTN 8"
- board text added: "BTN 9"
- board text added: "BTN10"
- board text added: "BTN11"
- board text added: "GND"
- board text added: "IO 1 - 8"
- board text added: "IO 9 - 16"
- board text added: "LED"
- board text added: "SERVO 1"
- board text added: "SERVO 2"
