File: Duck/duck_sensor.brd (EAGLE design)
At the start: 160 x 100 mm, 41 parts, among them J1 POWER_JACK, Q1 BC817-16LT1SMD, U1 MCP73831/OT, U2 DF04M, U3 MPU-9250DEV, U4 MCP6002, U5 BUZZER, X1 5268-02, X2 5267-03, X3 5268-02, X4 5268-02, X5 5268-02

Commit message: gerber
Parts:
- added C5, C6: 0.1uF, GFE:C0603(1608)_HANDSOLDER
- added D4: MMSZ5226B-7-F, GFE:SOD-123
- added H1, H2, H3, H4: MOUNT-HOLE3.2, holes:3,2
- added LOGO1: GRADEFREELOGO-20, GFE:GRADEFREELOGO-20
- added R17, R18, R21, R22, R24, R25: 1k, GFE:R0603(1608)_HANDSOLDER
- added R19, R20, R26, R27: 100k, GFE:R0603(1608)_HANDSOLDER
- added R23: 10k, GFE:R0603(1608)_HANDSOLDER
- added X10, X6, X7, X8, X9: 5268-02, GFE:5628-02
- C1: value 0.1uF -> 10uF, 16V; device GFE:C0603(1608)_HANDSOLDER -> berry:C1206(3216)-A
- C3: value 10uF, 16V -> 100uF, 16V; device berry:C1206(3216)-A -> adafruit:E2,5-6E
- J1: value POWER_JACK -> (none); device GFE:POWER_JACK_PTH -> SparkFun-Connectors:1X04
- J2: value (none) -> POWER_JACK; device SparkFun-Connectors:1X04 -> GFE:POWER_JACK_PTH
- JP1: value PARTICLE_PHOTONTEMPLATE -> JP2; device GFE:PARTICLE_PHOTON_TEMPLATE -> OSSI:JP2SMD0603
- JP2: value JP2 -> PARTICLE_PHOTONTEMPLATE; device OSSI:JP2SMD0603 -> GFE:PARTICLE_PHOTON_TEMPLATE
- R1, R5, R6: value 1k -> 4.7k
- R11: value 100k -> 1M
- R14: value 100k -> 10k
- R15, R16: value 10k -> 1k
- R2: value 2k -> 4.7k
- R3: value 4.7k -> 2k
- R4: value 4.7k -> 1k
- R7, R8: value 4.7k -> POT; device GFE:R0603(1608)_HANDSOLDER -> synth:RK09L
- U1: value MCP73831/OT -> MPU-9250DEV; device GFE:SOT23-5L -> GFE:MPU-9250
- U2: value DF04M -> MCP73831/OT; device GFE:DIL06 -> GFE:SOT23-5L
- U3: value MPU-9250DEV -> DF04M; device GFE:MPU-9250 -> GFE:DIL06
- U4: value MCP6002 -> BUZZER; device synth:DIL08 -> GFE:PS1240
- U5: value BUZZER -> MCP6002; device GFE:PS1240 -> synth:DIL08
- X1: value 5268-02 -> 5267-03; device GFE:5628-02 -> GFE:5267-03
- moved X5 383.0 mm to (29.2, 59.7), turned to 270 degrees
- moved D3 373.9 mm to (19.1, 40.6), turned to 180 degrees
- moved C4 370.8 mm to (-16.5, 73.7), turned to 270 degrees
- moved R16 365.5 mm to (-24.8, 34.3), turned to 180 degrees
- moved R15 353.6 mm to (-24.8, 52.1), turned to 180 degrees
- moved U4 352.2 mm to (-26.7, 73.7), turned to 270 degrees
- moved C3 344.8 mm to (30.5, 67.9)
- moved R13 327.3 mm to (33.0, 76.2), turned to 270 degrees
- moved U2 320.8 mm to (-11.4, 8.89), turned to 90 degrees
- moved R14 317.8 mm to (31.8, 72.4)
- moved JP2 299.6 mm to (0.00, 36.8), turned to 180 degrees
- moved R12 295.0 mm to (-18.4, 73.7), turned to 90 degrees
- moved C2 280.9 mm to (-7.62, 8.89), turned to 270 degrees
- moved X4 279.5 mm to (29.2, 41.9), turned to 270 degrees
- moved R11 261.0 mm to (19.1, 38.1)
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Connections:
- removed net N$16: JP1.19, JP1.D6
- removed net N$19: R13.1, R14.2
- removed net N$21: JP1.18, JP1.D5
- removed net N$22: JP1.15, JP1.D2
- removed net N$9: R10.1, R11.2
- removed net STRUT_GND: S1.G1, S1.G2, S1.G3, S1.G4
- new net A2: JP2.10, JP2.A2, R7.2
- new net A3: JP2.9, JP2.A3, R8.2
- new net A4: D3.C, JP2.8, JP2.A4, R11.2, R9.2
- new net N$23: C5.1, D4.C, R14.1, U5.3
- new net N$25: R21.2, X8.1
- new net N$26: R24.2, X8.2
- new net N$27: R22.2, X9.1
- new net N$28: C3.+, R13.2, R14.2, U3.4
- new net N$29: U3.1, X5.1
- new net N$30: U3.3, X5.2
- new net N$31: R25.2, X9.2
- new net PIXEL_LED: JP2.15, JP2.D2, X1.2
- new net S1: JP2.7, JP2.A5, R24.1, R26.2
- new net S2: JP2.18, JP2.D5, R17.1, R19.2
- new net S3: JP2.19, JP2.D6, R25.1, R27.2
- new net S4: JP2.20, JP2.D7, R18.1, R20.2
- new net VBAT_: JP2.22, JP2.VBAT_
- net 3.3V: now also C6.1, JP1.3, JP2.24, JP2.3V3, R1.1, R15.1, R16.1, R2.1, R21.1, R22.1, U1.VCC, U5.8, X10.1; no longer C4.1, JP1.24, JP1.3V3, JP2.3, R12.1, R9.1, U3.VCC, U4.8, X5.1
- net A0: now also JP2.12, JP2.A0, U5.6, U5.7; no longer U4.6, U4.7
- net A1: now also JP2.11, JP2.A1, U5.1, U5.2; no longer U4.1, U4.2
- net BUZZER_PWM: now also JP2.16, JP2.D3, R10.1; no longer JP1.16, JP1.D3, R5.1
- net GND: now also C3.-, C5.2, C6.2, D3.A, D4.A, J1.4, J2.GND, J2.GNDBREAK, JP2.2, JP2.21, JP2.GND@0, JP2.GND@2, R13.1, R19.1, R20.1, R23.1, R26.1, R27.1, R3.1, R7.3, R8.3, U1.GND, U2.2, U3.6, U5.4, X1.1, X3.2, X4.2; no longer C3.2, J1.GND, J1.GNDBREAK, J2.4, JP1.2, JP1.21, JP1.GND@0, JP1.GND@2, R14.1, R15.1, R2.1, U1.2, U3.GND, U4.4, X1.2
- net INT: now also JP2.17, JP2.D4, U1.INT; no longer JP1.17, JP1.D4, U3.INT
- net N$1: now also D2.C; no longer D1.C
- net N$10: now also R16.2, X7.1; no longer R12.2, X4.1
- net N$11: now also R18.2, X7.2; no longer R13.2, X4.2
- net N$12: now also JP2.3, JP2.TX, R5.2; no longer JP1.3, JP1.TX, R3.2
- net N$13: now also JP2.4, JP2.RX, R6.2; no longer JP1.4, JP1.RX, R4.2
- net N$14: now also R6.1; no longer R4.1
- net N$15: now also R5.1; no longer R3.1
- net N$17: now also R10.2; no longer R5.2
- net N$18: now also R12.1, U4.2; no longer R6.1, U5.2
- net N$2: now also R15.2, X6.1; no longer R9.2, X3.1
- net N$20: now also J1.1, JP1.2; no longer J2.1, JP2.2
- net N$24: now also R23.2, U5.5, X10.2; no longer R15.2, U4.5, X5.2
- net N$3: now also R4.2; no longer R1.2
- net N$4: now also U2.1; no longer U1.1
- net N$5: now also R3.2, U2.5; no longer R2.2, U1.5
- net N$6: now also D1.A, J2.PWR; no longer D2.A, J1.PWR
- net N$7: now also R9.1, X4.1; no longer JP1.20, JP1.D7
- net N$8: now also R17.2, X6.2; no longer R10.2, X3.2
- net SCL: now also J1.2, JP2.14, JP2.D1, R2.2, U1.SCL; no longer J2.2, JP1.14, JP1.D1, R7.2, U3.SCL
- net SDA: now also J1.3, JP2.13, JP2.D0, R1.2, U1.SDA; no longer J2.3, JP1.13, JP1.D0, R8.2, U3.SDA
- net VBAT: now also C2.1, D2.A, U2.3, X3.1; no longer C3.1, D1.A, JP1.22, JP1.VBAT, U1.3, X1.1
- net VIN: now also C4.1, D1.C, JP2.VIN, R12.2, R4.1, U2.4, U4.1, X1.3; no longer C2.1, D2.C, JP1.VIN, R1.1, R6.2, U1.4, U5.1
Routing:
- net 3.3V: track 0.00 -> 292.9 mm, vias 0 -> 10
- net VIN: track 0.00 -> 179.1 mm, vias 0 -> 7
- net A2: track 0.00 -> 55.6 mm, vias 0 -> 2
- net A1: track 0.00 -> 46.9 mm
- net GND: track 0.00 -> 39.6 mm, vias 0 -> 16
- net SCL: track 0.00 -> 39.1 mm
- net INT: track 0.00 -> 37.1 mm
- net A3: track 0.00 -> 36.7 mm, vias 0 -> 2
- net N$24: track 0.00 -> 36.3 mm, vias 0 -> 2
- net BUZZER_PWM: track 0.00 -> 33.9 mm, vias 0 -> 2
- net PIXEL_LED: track 0.00 -> 28.9 mm
- net SDA: track 0.00 -> 28.9 mm
- net A0: track 0.00 -> 28.0 mm
- net N$1: track 0.00 -> 25.8 mm
- net N$28: track 0.00 -> 25.0 mm
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- added copper zone on layer 16, net GND
Other:
- board size 160 x 100 mm -> 72 x 102 mm
