File: Duck/duck_sensor.sch (EAGLE design)
At the start: 41 parts, among them J1 POWER_JACK, Q1 BC817-16LT1SMD, U1 MCP73831/OT, U2 DF04M, U3 MPU-9250DEV, U4 MCP6002, U5 BUZZER, X1 5268-02, X2 5267-03, X3 5268-02, X4 5268-02, X5 5268-02

Commit message: gerber
Parts:
- added C5, C6: 0.1uF, GFE:C0603(1608)_HAND
- added D4: MMSZ5226B-7-F, GFE:MMSZ5226B-7-F
- added H1, H2, H3, H4: MOUNT-HOLE3.2, holes:MOUNT-HOLE3.2
- added LOGO1: GRADEFREELOGO-20, GFE:GRADEFREELOGO-20
- added R17, R18, R21, R22, R24, R25: 1k, GFE:R0603(1608)_HAND
- added R19, R20, R26, R27: 100k, GFE:R0603(1608)_HAND
- added R23: 10k, GFE:R0603(1608)_HAND
- added X10, X6, X7, X8, X9: 5268-02, GFE:5268-02
- C1: value 0.1uF -> 10uF, 16V; device GFE:C0603(1608)_HAND -> berry:C-TANTAL-A
- C3: value 10uF, 16V -> 100uF, 16V; device berry:C-TANTAL-A -> adafruit:CPOL-USE2,5-6E
- J1: value POWER_JACK -> (none); device GFE:POWER_JACK -> SparkFun-Connectors:CONN_04
- J2: value (none) -> POWER_JACK; device SparkFun-Connectors:CONN_04 -> GFE:POWER_JACK
- JP1: value PARTICLE_PHOTONTEMPLATE -> JP2; device GFE:PARTICLE_PHOTONTEMPLATE -> OSSI:JP2
- JP2: value JP2 -> PARTICLE_PHOTONTEMPLATE; device OSSI:JP2 -> GFE:PARTICLE_PHOTONTEMPLATE
- R1, R5, R6: value 1k -> 4.7k
- R11: value 100k -> 1M
- R14: value 100k -> 10k
- R15, R16: value 10k -> 1k
- R2: value 2k -> 4.7k
- R3: value 4.7k -> 2k
- R4: value 4.7k -> 1k
- R7, R8: value 4.7k -> POT; device GFE:R0603(1608)_HAND -> synth:POT
- U1: value MCP73831/OT -> MPU-9250DEV; device GFE:MCP73831/OT -> GFE:MPU-9250DEV
- U2: value DF04M -> MCP73831/OT; device GFE:DF04M -> GFE:MCP73831/OT
- U3: value MPU-9250DEV -> DF04M; device GFE:MPU-9250DEV -> GFE:DF04M
- U4: value MCP6002 -> BUZZER; device synth:MCP6002 -> GFE:BUZZER
- U5: value BUZZER -> MCP6002; device GFE:BUZZER -> synth:MCP6002
- X1: value 5268-02 -> 5267-03; device GFE:5268-02 -> GFE:5267-03
Connections:
- removed net N$16: JP1.(JTAG_TCK)D6
- removed net N$19: R13.1, R14.2
- removed net N$21: JP1.(JTAG_TDI)D5
- removed net N$22: JP1.D2
- removed net N$9: R10.1, R11.2
- removed net STRUT_GND: S1.GNDTERMINAL, S1.GNDTERMINAL1, S1.GNDTERMINAL2, S1.GNDTERMINAL3
- new net A2: JP2.A2(SPI1_SS), R7.S
- new net A3: JP2.A3(SPI1_SCK), R8.S
- new net A4: D3.C, JP2.A4(SPI1_MISO), R11.2, R9.2
- new net N$23: C5.1, D4.C, R14.1, U5A.+IN
- new net N$25: R21.2, X8.1
- new net N$26: R24.2, X8.2
- new net N$27: R22.2, X9.1
- new net N$28: C3.+, R13.2, R14.2, U3.+
- new net N$29: U3.P$1, X5.1
- new net N$30: U3.P$2, X5.2
- new net N$31: R25.2, X9.2
- new net PIXEL_LED: JP2.D2, X1.2
- new net S1: JP2.A5(SPI1_MOSI), R24.1, R26.2
- new net S2: JP2.(JTAG_TDI)D5, R17.1, R19.2
- new net S3: JP2.(JTAG_TCK)D6, R25.1, R27.2
- new net S4: JP2.(JTAG_TMS)D7, R18.1, R20.2
- net 3.3V: now also C6.1, JP1.3, JP2.+3V3, R1.1, R15.1, R16.1, R2.1, R21.1, R22.1, R7.E, R8.E, U1.VCC, U5G$3.V+, X10.1; no longer C4.1, JP1.+3V3, JP2.3, R12.1, R7.1, R8.1, R9.1, U3.VCC, U4G$3.V+, X5.1
- net A0: now also JP2.A0, U5B.-IN, U5B.OUT; no longer U4B.-IN, U4B.OUT
- net A1: now also JP2.A1, U5A.-IN, U5A.OUT; no longer U4A.-IN, U4A.OUT
- net BUZZER_PWM: now also JP2.(JTAG_TRST)D3, R10.1; no longer JP1.(JTAG_TRST)D3, R5.1
- net GND: now also C1.-, C5.2, C6.2, D3.A, D4.A, J1.4, J2.GND, J2.GNDBREAK, JP2.GND@2, JP2.GND@21, R13.1, R19.1, R20.1, R23.1, R26.1, R27.1, R3.1, R7.A, R8.A, U1.GND, U2.VSS, U3.-, U5G$3.V-, X1.1, X3.2, X4.2; no longer C1.2, J1.GND, J1.GNDBREAK, J2.4, JP1.GND@2, JP1.GND@21, R14.1, R15.1, R2.1, U1.VSS, U3.GND, U4G$3.V-, X1.2
- net INT: now also JP2.(JTAG_TDO)D4, U1.INT; no longer JP1.(JTAG_TDO)D4, U3.INT
- net N$1: now also D2.C; no longer D1.C
- net N$10: now also R16.2, X7.1; no longer R12.2, X4.1
- net N$11: now also R18.2, X7.2; no longer R13.2, X4.2
- net N$12: now also JP2.TX, R5.2; no longer JP1.TX, R3.2
- net N$13: now also JP2.RX, R6.2; no longer JP1.RX, R4.2
- net N$14: now also R6.1; no longer R4.1
- net N$15: now also R5.1; no longer R3.1
- net N$17: now also R10.2; no longer R5.2
- net N$18: now also R12.1, U4.P$2; no longer R6.1, U5.P$2
- net N$2: now also R15.2, X6.1; no longer R9.2, X3.1
- net N$20: now also J1.1, JP1.2; no longer J2.1, JP2.2
- net N$24: now also R23.2, U5B.+IN, X10.2; no longer R15.2, U4B.+IN, X5.2
- net N$3: now also R4.2; no longer R1.2
- net N$4: now also U2.STAT; no longer U1.STAT
- net N$5: now also R3.2, U2.PROG; no longer R2.2, U1.PROG
- net N$6: now also D1.A, J2.PWR; no longer D2.A, J1.PWR
- net N$7: now also R9.1, X4.1; no longer JP1.(JTAG_TMS)D7
- net N$8: now also R17.2, X6.2; no longer R10.2, X3.2
- net SCL: now also J1.2, JP2.(SCL)D1, R2.2, U1.SCL; no longer J2.2, JP1.(SCL)D1, R7.2, U3.SCL
- net SDA: now also J1.3, JP2.(SDA)D0, R1.2, U1.SDA; no longer J2.3, JP1.(SDA)D0, R8.2, U3.SDA
- net VBAT: now also C2.+, D2.A, U2.VBAT, X3.1; no longer C3.+, D1.A, U1.VBAT, X1.1
- net VIN: now also C1.+, C4.1, D1.C, JP1.1, JP2.VIN, R12.2, R4.1, U2.VDD, U4.P$1, X1.3; no longer C1.1, C2.+, D2.C, JP1.VIN, JP2.1, R1.1, R6.2, U1.VDD, U5.P$1
Other:
- note added: "piezo interface"
- moved on the sheet: C2, C3, C4, D1, D2, D3, R1, R10, R11, R12, R13, R14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

Commit message: comment
Other:
- note added: "Tear / Water / Resistive Fluid to Analog Input"
- note added: "touch"
Changed lines of the file:
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@@
 <text x="96.52" y="96.52" size="1.778" layer="91" rot="R180">PullUp R is already in MPU-9250 Dev</text>
 <text x="190.5" y="10.16" size="1.778" layer="91">piezo interface</text>
+<text x="307.34" y="132.08" size="1.778" layer="91">Tear / Water / Resistive Fluid to Analog Input</text>
+<text x="241.3" y="129.54" size="1.778" layer="91">touch</text>
+<text x="241.3" y="86.36" size="1.778" layer="91">touch</text>
+<text x="312.42" y="86.36" size="1.778" layer="91">touch</text>
 </plain>
 <instances>

Commit message: comment added
Other:
- note added: "3.3V zener for overvoltage protection"
- note added: "select exter i2c power"
- moved on the sheet: H1, H2, H3, H4
Changed lines of the file:
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@@
 <text x="241.3" y="86.36" size="1.778" layer="91">touch</text>
 <text x="312.42" y="86.36" size="1.778" layer="91">touch</text>
+<text x="190.5" y="5.08" size="1.778" layer="91">3.3V zener for overvoltage protection</text>
+<text x="243.84" y="210.82" size="1.778" layer="91">3.3V zener for overvoltage protection</text>
+<text x="7.62" y="27.94" size="1.778" layer="91">select exter i2c power</text>
 </plain>
 <instances>
@@
 <instance part="VIN2" gate="G$1" x="20.32" y="116.84" rot="R90"/>
 <instance part="LOGO1" gate="G$1" x="144.78" y="134.62"/>
-<instance part="H1" gate="G$1" x="299.72" y="165.1"/>
-<instance part="H2" gate="G$1" x="330.2" y="167.64"/>
-<instance part="H3" gate="G$1" x="363.22" y="167.64"/>
-<instance part="H4" gate="G$1" x="373.38" y="152.4"/>
+<instance part="H1" gate="G$1" x="271.78" y="165.1"/>
+<instance part="H2" gate="G$1" x="302.26" y="165.1"/>
+<instance part="H3" gate="G$1" x="271.78" y="154.94"/>
+<instance part="H4" gate="G$1" x="302.26" y="154.94"/>
 </instances>
 <busses>

Commit message: comment
Other:
- note added: "D4 is for LED!!! S4 is not being used now"
Changed lines of the file:
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@@
 <text x="243.84" y="210.82" size="1.778" layer="91">3.3V zener for overvoltage protection</text>
 <text x="7.62" y="27.94" size="1.778" layer="91">select exter i2c power</text>
+<text x="236.22" y="45.72" size="1.778" layer="91">D4 is for LED!!! S4 is not being used now</text>
 </plain>
 <instances>
